File: 6502_6802 Board v2/schematic/CPU6502_6802/CPU6502_6802.kicad_pcb (KiCad board)
At the start: 2 copper layers, 100 x 100 mm, 67 parts, among them J1 BUS, J10 Conn_01x01, J11 Conn_01x01, J12 Conn_01x01, J13 Conn_01x01, J14 Conn_01x01, J15 Conn_01x01, J2 BUS, J20 Conn_01x12, J21 Conn_01x12, J22 Conn_02x36_Counter_Clockwise, J23 Conn_02x36_Counter_Clockwise, J24 Conn_02x36_Counter_Clockwise, J25 Conn_02x36_Counter_Clockwise, J26 Conn_02x36_Counter_Clockwise, J3 BUS, J30 Conn_01x06, J31 Conn_01x06, J4 BUS, J5 Conn_01x09, J6 Conn_01x08, J7 Conn_01x08, J8 Conn_01x09, J9 Conn_02x05_Odd_Even, U1 XC9572VQ44, U2 SN74LVC245ANSR, U3 SN74LVC245ANSR, U5 SN74LVCC3245ANSR, U6 SN74LVC245ANSR, U7 W65C02SxP, U8 SN74LVC125AD, U9 SN74LVC125AD

Commit message: Readme update
Parts:
- R10, R11, R9: value 10k -> 1k
Changed lines of the file:
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@@
         (effects (font (size 1 1) (thickness 0.15)) (justify mirror))
     )
-    (fp_text value "10k" (at 0 -1.82 90) (layer "B.Fab")
+    (fp_text value "1k" (at 0 -1.82 90) (layer "B.Fab")
         (effects (font (size 1 1) (thickness 0.15)) (justify mirror))
     )
@@
         (effects (font (size 1 1) (thickness 0.15)) (justify mirror))
     )
-    (fp_text value "10k" (at 0 -1.82) (layer "B.Fab")
+    (fp_text value "1k" (at 0 -1.82) (layer "B.Fab")
         (effects (font (size 1 1) (thickness 0.15)) (justify mirror))
     )
@@
         (effects (font (size 1 1) (thickness 0.15)) (justify mirror))
     )
-    (fp_text value "10k" (at 0 -1.82) (layer "B.Fab")
-        (effects (font (size 1 1) (thickness 0.15)) (justify mirror))
-    )
+    (fp_text value "1k" (at 0 -1.82) (layer "B.Fab")
+        (effects (font (size 1 1) (thickness 0.15)) (justify mirror))
+    )
