File: 6502_6802 Board v2/schematic/CPU6502_6802/CPU6502_6802.kicad_pcb (KiCad board)
At the start: 2 copper layers, 100 x 100 mm, 67 parts, among them J1 BUS, J10 Conn_01x01, J11 Conn_01x01, J12 Conn_01x01, J13 Conn_01x01, J14 Conn_01x01, J15 Conn_01x01, J2 BUS, J20 Conn_01x12, J21 Conn_01x12, J22 Conn_02x36_Counter_Clockwise, J23 Conn_02x36_Counter_Clockwise, J24 Conn_02x36_Counter_Clockwise, J25 Conn_02x36_Counter_Clockwise, J26 Conn_02x36_Counter_Clockwise, J3 BUS, J30 Conn_01x06, J31 Conn_01x06, J4 BUS, J5 Conn_01x09, J6 Conn_01x08, J7 Conn_01x08, J8 Conn_01x09, J9 Conn_02x05_Odd_Even, U1 XC9572VQ44, U2 SN74LVC245ANSR, U3 SN74LVC245ANSR, U5 SN74LVCC3245ANSR, U6 SN74LVC245ANSR, U7 W65C02SxP, U8 SN74LVC125AD, U9 SN74LVC125AD

Commit message: DREAM6800 video started
Parts:
- added JP9: PH2_5/8, Jumper:SolderJumper-3_P1.3mm_Open_RoundedPad1.0x1.5mm_NumberLabels, F.Cu at (135.0, 76.0)
- added R12: 10k, Resistor_SMD:R_1206_3216Metric_Pad1.30x1.75mm_HandSolder, B.Cu at (173.9, 111.6)
Connections:
- net /IO1 renamed /E_OUT
- J5 pad 4: /A0 -> /HALT_in
- J7 pad 7: /IO2 -> /RDY
- J7 pad 8: /IO3 -> /SYNC
- U1 pad 30: /A0 -> /HALT_in
- U1 pad 41: /IO2 -> /RDY
- U1 pad 42: /IO3 -> /SYNC
- U9 pad 2: /PHI2 -> /Buffers/PHI2
Routing:
- net /A0: track 113.8 -> 23.7 mm
- net /E_OUT: track 5.68 -> 83.1 mm, vias 0 -> 3
- net /RDY: track 48.5 -> 101.6 mm, vias 0 -> 1
- net /SYNC: track 64.9 -> 106.3 mm, vias 0 -> 1
- net /R/~{W}: track 70.8 -> 60.2 mm
- net /HALT_in: track 0.00 -> 10.4 mm
- net /IO3: track 9.03 -> 0.00 mm
- net /IO2: track 7.18 -> 0.00 mm
- net +3V3: track 210.8 -> 217.1 mm
- net /PHI2: track 75.2 -> 70.7 mm
- net /Buffers/PHI2: track 0.00 -> 3.04 mm
- net /~{NMI}: track 56.2 -> 53.3 mm, vias 0 -> 1
- net /~{ML}: track 91.1 -> 93.3 mm
- net /Buffers/VBuffer: track 188.4 -> 189.9 mm
- net /PHI1: track 89.5 -> 88.4 mm
