File: 6502_6802 Board v2/schematic/CPU6502_6802/buffers.kicad_sch (KiCad schematic)
At the start: 23 parts, among them J10 Conn_01x01, J11 Conn_01x01, J12 Conn_01x01, J13 Conn_01x01, J14 Conn_01x01, J15 Conn_01x01, J30 Conn_01x06, J31 Conn_01x06, U5 SN74LVCC3245ANSR, U8 SN74LVC125AD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

Commit message: Readme update
Parts:
- R10, R11, R9: value 10k -> 1k
Other:
- note added: "maybe consider ~{MWR} and ~{MRD} NOT High-Z with AOE. Is this really necessary?"
Changed lines of the file:
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@@
     (stroke (width 0) (type default))
+  )
+  (text "maybe consider ~{MWR} and ~{MRD}\nNOT High-Z with AOE. \nIs this really necessary?"
+    (at 170.18 160.655 0)
+    (effects (font (size 1.27 1.27)) (justify left bottom))
   )
   (text "One can place a SN74LVC245ANSR for 3.3V BUS and CPU or\na SN74ABT245BNSR for 5V BUS and CPU on the Pads from U5\nor leave the SN74LVCC3245ANSR for 3.3V BUS and 5V CPU.\n"
@@
   (symbol (lib_id "Device:R_Small") (at 196.85 137.795 0) (unit 1)
     (in_bom yes) (on_board yes) (dnp no) (fields_autoplaced)
-    (property "Reference" "R11" (at 198.3486 136.771 0)
-      (effects (font (size 1.27 1.27)) (justify left))
-    )
-    (property "Value" "10k" (at 198.3486 138.819 0)
+    (property "Reference" "R11" (at 198.3486 136.5829 0)
+      (effects (font (size 1.27 1.27)) (justify left))
+    )
+    (property "Value" "1k" (at 198.3486 139.0071 0)
       (effects (font (size 1.27 1.27)) (justify left))
     )
@@
   (symbol (lib_id "Device:R_Small") (at 196.85 97.79 0) (unit 1)
     (in_bom yes) (on_board yes) (dnp no) (fields_autoplaced)
-    (property "Reference" "R9" (at 198.3486 96.766 0)
-      (effects (font (size 1.27 1.27)) (justify left))
-    )
-    (property "Value" "10k" (at 198.3486 98.814 0)
+    (property "Reference" "R9" (at 198.3486 96.5779 0)
+      (effects (font (size 1.27 1.27)) (justify left))
+    )
+    (property "Value" "1k" (at 198.3486 99.0021 0)
       (effects (font (size 1.27 1.27)) (justify left))
     )
@@
   (symbol (lib_id "Device:R_Small") (at 196.215 116.205 0) (unit 1)
     (in_bom yes) (on_board yes) (dnp no) (fields_autoplaced)
-    (property "Reference" "R10" (at 197.7136 115.181 0)
-      (effects (font (size 1.27 1.27)) (justify left))
-    )
-    (property "Value" "10k" (at 197.7136 117.229 0)
-      (effects (font (size 1.27 1.27)) (justify left))
-    )
+    (property "Reference" "R10" (at 197.7136 114.9929 0)
+      (effects (font (size 1.27 1.27)) (justify left))
+    )
+    (property "Value" "1k" (at 197.7136 117.4171 0)
+      (effects (font (size 1.27 1.27)) (justify left))
+    )
