File: 6502_6802 Board v2/schematic/CPU6502_6802/bus.kicad_sch (KiCad schematic)
At the start: 6 parts

Commit message: Readme update
Connections:
- net RX2: now also J?.3 (Pin_3), J?.3 (Pin_3); no longer J?.4 (Pin_4), J?.4 (Pin_4)
- net RX3: now also J?.5 (Pin_5), J?.5 (Pin_5); no longer J?.6 (Pin_6), J?.6 (Pin_6)
- net TX2: now also J?.4 (Pin_4), J?.4 (Pin_4); no longer J?.3 (Pin_3), J?.3 (Pin_3)
- net TX3: now also J?.6 (Pin_6), J?.6 (Pin_6); no longer J?.5 (Pin_5), J?.5 (Pin_5)
Changed lines of the file:
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@@
     (effects (font (size 1.27 1.27)) (justify right bottom))
   )
-  (label "RX3" (at 100.965 96.52 180) (fields_autoplaced)
-    (effects (font (size 1.27 1.27)) (justify right bottom))
+  (label "RX3" (at 62.865 96.52 0) (fields_autoplaced)
+    (effects (font (size 1.27 1.27)) (justify left bottom))
   )
   (label "A15" (at 156.21 67.31 180) (fields_autoplaced)
@@
     (effects (font (size 1.27 1.27)) (justify left bottom))
   )
-  (label "TX3" (at 62.865 96.52 0) (fields_autoplaced)
-    (effects (font (size 1.27 1.27)) (justify left bottom))
+  (label "TX3" (at 100.965 96.52 180) (fields_autoplaced)
+    (effects (font (size 1.27 1.27)) (justify right bottom))
   )
   (label "D3" (at 39.37 95.885 180) (fields_autoplaced)
@@
     (effects (font (size 1.27 1.27)) (justify right bottom))
   )
-  (label "RX2" (at 100.965 93.98 180) (fields_autoplaced)
-    (effects (font (size 1.27 1.27)) (justify right bottom))
+  (label "RX2" (at 62.865 93.98 0) (fields_autoplaced)
+    (effects (font (size 1.27 1.27)) (justify left bottom))
   )
   (label "A3" (at 156.21 52.07 180) (fields_autoplaced)
@@
     (effects (font (size 1.27 1.27)) (justify right bottom))
   )
-  (label "TX2" (at 62.865 93.98 0) (fields_autoplaced)
-    (effects (font (size 1.27 1.27)) (justify left bottom))
+  (label "TX2" (at 100.965 93.98 180) (fields_autoplaced)
+    (effects (font (size 1.27 1.27)) (justify right bottom))
   )
   (label "A5" (at 104.14 54.61 180) (fields_autoplaced)
@@
     (effects (font (size 1.27 1.27)) (justify right))
   )
-  (hierarchical_label "RX2" (shape input) (at 161.925 93.98 0) (fields_autoplaced)
-    (effects (font (size 1.27 1.27)) (justify left))
+  (hierarchical_label "RX2" (shape input) (at 122.555 93.98 180) (fields_autoplaced)
+    (effects (font (size 1.27 1.27)) (justify right))
   )
   (hierarchical_label "TDO" (shape output) (at 156.845 132.08 0) (fields_autoplaced)
@@
     (effects (font (size 1.27 1.27)) (justify right))
   )
-  (hierarchical_label "TX2" (shape output) (at 122.555 93.98 180) (fields_autoplaced)
-    (effects (font (size 1.27 1.27)) (justify right))
+  (hierarchical_label "TX2" (shape output) (at 161.925 93.98 0) (fields_autoplaced)
+    (effects (font (size 1.27 1.27)) (justify left))
   )
   (hierarchical_label "~{PH0}" (shape output) (at 161.925 104.14 0) (fields_autoplaced)
@@
     (effects (font (size 1.27 1.27)) (justify right))
   )
-  (hierarchical_label "TX3" (shape input) (at 122.555 96.52 180) (fields_autoplaced)
-    (effects (font (size 1.27 1.27)) (justify right))
+  (hierarchical_label "TX3" (shape output) (at 161.925 96.52 0) (fields_autoplaced)
+    (effects (font (size 1.27 1.27)) (justify left))
   )
   (hierarchical_label "SCK" (shape output) (at 127 129.54 180) (fields_autoplaced)
@@
     (effects (font (size 1.27 1.27)) (justify left))
   )
-  (hierarchical_label "RX3" (shape input) (at 161.925 96.52 0) (fields_autoplaced)
-    (effects (font (size 1.27 1.27)) (justify left))
+  (hierarchical_label "RX3" (shape input) (at 122.555 96.52 180) (fields_autoplaced)
+    (effects (font (size 1.27 1.27)) (justify right))
   )
   (hierarchical_label "PHI2_e" (shape output) (at 151.13 29.21 0) (fields_autoplaced)

Commit message: Z80 added
Parts:
- gave numbers to parts that had none: 4
