File: 6809_Board/CPU_6809_board/CPU_6809_board.kicad_sch (KiCad schematic)
At the start: 33 parts, among them J5 Conn_01x09, J6 Conn_01x08, J7 Conn_01x08, J8 Conn_01x09, J9 Conn_02x05_Odd_Even, U1 XC9572VQ44, U22 MC6809E, U23 MC6809

Commit message: Readme update
Changed lines of the file:
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@@
     (effects (font (size 1.27 1.27)) (justify left bottom))
   )
-  (label "TX2" (at 14.605 46.355 0) (fields_autoplaced)
+  (label "TX2" (at 14.605 43.815 0) (fields_autoplaced)
     (effects (font (size 1.27 1.27)) (justify left bottom))
   )
@@
     (effects (font (size 1.27 1.27)) (justify right bottom))
   )
-  (label "TX3" (at 14.605 51.435 0) (fields_autoplaced)
+  (label "TX3" (at 14.605 48.895 0) (fields_autoplaced)
     (effects (font (size 1.27 1.27)) (justify left bottom))
   )
@@
     (effects (font (size 1.27 1.27)) (justify right bottom))
   )
-  (label "RX3" (at 14.605 48.895 0) (fields_autoplaced)
+  (label "RX3" (at 14.605 51.435 0) (fields_autoplaced)
     (effects (font (size 1.27 1.27)) (justify left bottom))
   )
@@
     (effects (font (size 1.27 1.27)) (justify left bottom))
   )
-  (label "RX2" (at 14.605 43.815 0) (fields_autoplaced)
-    (effects (font (size 1.27 1.27)) (justify left bottom))
-  )
+  (label "RX2" (at 14.605 46.355 0) (fields_autoplaced)
+    (effects (font (size 1.27 1.27)) (justify left bottom))
+  )
