File: Fill_Memory_Board/Fill_Memory_Board.kicad_pcb (KiCad board)
At the start: 2 copper layers, 100 x 100 mm, 43 parts, among them J1 BUS, J2 BUS, J20 Conn_01x32, J21 Conn_01x32, J22 Conn_01x38, J23 Conn_01x38, J24 Conn_01x38, J25 Conn_01x38, J26 Conn_01x38, J27 Conn_01x38, J28 Conn_01x38, J29 Conn_01x38, J3 BUS, J30 Conn_01x38, J31 Conn_01x38, J32 Conn_01x32, J4 BUS, J6 STM32F411, Q1 PMV450ENEAR, U1 74LS125, U10 74LVC595, U12 74AHC1G14, U16 74LVC138, U17 74LVC138, U18 74HC590, U19 74HC590, U20 74HC590, U9 74LS165

Commit message: Readme update
Connections:
- J20 pad 10: (no net) -> unconnected-(J20-Pin_10-Pad10)
- J20 pad 11: (no net) -> unconnected-(J20-Pin_11-Pad11)
- J20 pad 12: (no net) -> unconnected-(J20-Pin_12-Pad12)
- J20 pad 13: (no net) -> unconnected-(J20-Pin_13-Pad13)
- J20 pad 14: (no net) -> unconnected-(J20-Pin_14-Pad14)
- J20 pad 15: (no net) -> unconnected-(J20-Pin_15-Pad15)
- J20 pad 16: (no net) -> unconnected-(J20-Pin_16-Pad16)
- J20 pad 17: (no net) -> unconnected-(J20-Pin_17-Pad17)
- J20 pad 18: (no net) -> unconnected-(J20-Pin_18-Pad18)
- J20 pad 19: (no net) -> unconnected-(J20-Pin_19-Pad19)
- J20 pad 2: (no net) -> unconnected-(J20-Pin_2-Pad2)
- J20 pad 20: (no net) -> unconnected-(J20-Pin_20-Pad20)
- J20 pad 21: (no net) -> unconnected-(J20-Pin_21-Pad21)
- J20 pad 22: (no net) -> unconnected-(J20-Pin_22-Pad22)
- J20 pad 23: (no net) -> unconnected-(J20-Pin_23-Pad23)
- J20 pad 24: (no net) -> unconnected-(J20-Pin_24-Pad24)
- J20 pad 25: (no net) -> unconnected-(J20-Pin_25-Pad25)
- J20 pad 26: (no net) -> unconnected-(J20-Pin_26-Pad26)
- J20 pad 27: (no net) -> unconnected-(J20-Pin_27-Pad27)
- J20 pad 28: (no net) -> unconnected-(J20-Pin_28-Pad28)
- J20 pad 29: (no net) -> unconnected-(J20-Pin_29-Pad29)
- J20 pad 3: (no net) -> unconnected-(J20-Pin_3-Pad3)
- J20 pad 30: (no net) -> unconnected-(J20-Pin_30-Pad30)
- J20 pad 31: (no net) -> unconnected-(J20-Pin_31-Pad31)
- J20 pad 4: (no net) -> unconnected-(J20-Pin_4-Pad4)
- J20 pad 5: (no net) -> unconnected-(J20-Pin_5-Pad5)
- J20 pad 6: (no net) -> unconnected-(J20-Pin_6-Pad6)
- J20 pad 7: (no net) -> unconnected-(J20-Pin_7-Pad7)
- J20 pad 8: (no net) -> unconnected-(J20-Pin_8-Pad8)
- J20 pad 9: (no net) -> unconnected-(J20-Pin_9-Pad9)
- J21 pad 10: (no net) -> unconnected-(J21-Pin_10-Pad10)
- J21 pad 11: (no net) -> unconnected-(J21-Pin_11-Pad11)
- J21 pad 12: (no net) -> unconnected-(J21-Pin_12-Pad12)
- J21 pad 13: (no net) -> unconnected-(J21-Pin_13-Pad13)
- J21 pad 14: (no net) -> unconnected-(J21-Pin_14-Pad14)
- J21 pad 15: (no net) -> unconnected-(J21-Pin_15-Pad15)
- J21 pad 16: (no net) -> unconnected-(J21-Pin_16-Pad16)
- J21 pad 17: (no net) -> unconnected-(J21-Pin_17-Pad17)
- J21 pad 18: (no net) -> unconnected-(J21-Pin_18-Pad18)
- J21 pad 19: (no net) -> unconnected-(J21-Pin_19-Pad19)
- J21 pad 2: (no net) -> unconnected-(J21-Pin_2-Pad2)
- J21 pad 20: (no net) -> unconnected-(J21-Pin_20-Pad20)
- J21 pad 21: (no net) -> unconnected-(J21-Pin_21-Pad21)
- J21 pad 22: (no net) -> unconnected-(J21-Pin_22-Pad22)
- J21 pad 23: (no net) -> unconnected-(J21-Pin_23-Pad23)
- J21 pad 24: (no net) -> unconnected-(J21-Pin_24-Pad24)
- J21 pad 25: (no net) -> unconnected-(J21-Pin_25-Pad25)
- J21 pad 26: (no net) -> unconnected-(J21-Pin_26-Pad26)
- J21 pad 27: (no net) -> unconnected-(J21-Pin_27-Pad27)
- J21 pad 28: (no net) -> unconnected-(J21-Pin_28-Pad28)
- J21 pad 29: (no net) -> unconnected-(J21-Pin_29-Pad29)
- J21 pad 3: (no net) -> unconnected-(J21-Pin_3-Pad3)
- J21 pad 30: (no net) -> unconnected-(J21-Pin_30-Pad30)
- J21 pad 31: (no net) -> unconnected-(J21-Pin_31-Pad31)
- J21 pad 4: (no net) -> unconnected-(J21-Pin_4-Pad4)
- J21 pad 5: (no net) -> unconnected-(J21-Pin_5-Pad5)
- J21 pad 6: (no net) -> unconnected-(J21-Pin_6-Pad6)
- J21 pad 7: (no net) -> unconnected-(J21-Pin_7-Pad7)
- J21 pad 8: (no net) -> unconnected-(J21-Pin_8-Pad8)
- J21 pad 9: (no net) -> unconnected-(J21-Pin_9-Pad9)
- J22 pad 10: (no net) -> unconnected-(J22-Pin_10-Pad10)
- J22 pad 11: (no net) -> unconnected-(J22-Pin_11-Pad11)
- J22 pad 12: (no net) -> unconnected-(J22-Pin_12-Pad12)
- J22 pad 13: (no net) -> unconnected-(J22-Pin_13-Pad13)
- J22 pad 14: (no net) -> unconnected-(J22-Pin_14-Pad14)
- J22 pad 15: (no net) -> unconnected-(J22-Pin_15-Pad15)
- J22 pad 16: (no net) -> unconnected-(J22-Pin_16-Pad16)
- J22 pad 17: (no net) -> unconnected-(J22-Pin_17-Pad17)
- J22 pad 18: (no net) -> unconnected-(J22-Pin_18-Pad18)
- J22 pad 19: (no net) -> unconnected-(J22-Pin_19-Pad19)
- J22 pad 20: (no net) -> unconnected-(J22-Pin_20-Pad20)
- J22 pad 21: (no net) -> unconnected-(J22-Pin_21-Pad21)
- J22 pad 22: (no net) -> unconnected-(J22-Pin_22-Pad22)
- J22 pad 23: (no net) -> unconnected-(J22-Pin_23-Pad23)
- J22 pad 24: (no net) -> unconnected-(J22-Pin_24-Pad24)
- J22 pad 25: (no net) -> unconnected-(J22-Pin_25-Pad25)
- J22 pad 26: (no net) -> unconnected-(J22-Pin_26-Pad26)
- J22 pad 27: (no net) -> unconnected-(J22-Pin_27-Pad27)
- J22 pad 28: (no net) -> unconnected-(J22-Pin_28-Pad28)
- J22 pad 29: (no net) -> unconnected-(J22-Pin_29-Pad29)
- J22 pad 3: (no net) -> unconnected-(J22-Pin_3-Pad3)
- J22 pad 30: (no net) -> unconnected-(J22-Pin_30-Pad30)
- J22 pad 31: (no net) -> unconnected-(J22-Pin_31-Pad31)
- J22 pad 32: (no net) -> unconnected-(J22-Pin_32-Pad32)
- J22 pad 33: (no net) -> unconnected-(J22-Pin_33-Pad33)
- J22 pad 34: (no net) -> unconnected-(J22-Pin_34-Pad34)
- J22 pad 35: (no net) -> unconnected-(J22-Pin_35-Pad35)
- J22 pad 36: (no net) -> unconnected-(J22-Pin_36-Pad36)
- J22 pad 37: (no net) -> unconnected-(J22-Pin_37-Pad37)
- J22 pad 4: (no net) -> unconnected-(J22-Pin_4-Pad4)
- J22 pad 5: (no net) -> unconnected-(J22-Pin_5-Pad5)
- J22 pad 6: (no net) -> unconnected-(J22-Pin_6-Pad6)
- J22 pad 7: (no net) -> unconnected-(J22-Pin_7-Pad7)
- J22 pad 8: (no net) -> unconnected-(J22-Pin_8-Pad8)
- J22 pad 9: (no net) -> unconnected-(J22-Pin_9-Pad9)
- J23 pad 10: (no net) -> unconnected-(J23-Pin_10-Pad10)
- J23 pad 11: (no net) -> unconnected-(J23-Pin_11-Pad11)
- J23 pad 12: (no net) -> unconnected-(J23-Pin_12-Pad12)
- J23 pad 13: (no net) -> unconnected-(J23-Pin_13-Pad13)
- J23 pad 14: (no net) -> unconnected-(J23-Pin_14-Pad14)
- J23 pad 15: (no net) -> unconnected-(J23-Pin_15-Pad15)
- J23 pad 16: (no net) -> unconnected-(J23-Pin_16-Pad16)
- J23 pad 17: (no net) -> unconnected-(J23-Pin_17-Pad17)
- J23 pad 18: (no net) -> unconnected-(J23-Pin_18-Pad18)
- J23 pad 19: (no net) -> unconnected-(J23-Pin_19-Pad19)
- J23 pad 20: (no net) -> unconnected-(J23-Pin_20-Pad20)
- J23 pad 21: (no net) -> unconnected-(J23-Pin_21-Pad21)
- J23 pad 22: (no net) -> unconnected-(J23-Pin_22-Pad22)
- J23 pad 23: (no net) -> unconnected-(J23-Pin_23-Pad23)
- J23 pad 24: (no net) -> unconnected-(J23-Pin_24-Pad24)
- J23 pad 25: (no net) -> unconnected-(J23-Pin_25-Pad25)
- J23 pad 26: (no net) -> unconnected-(J23-Pin_26-Pad26)
- J23 pad 27: (no net) -> unconnected-(J23-Pin_27-Pad27)
- J23 pad 28: (no net) -> unconnected-(J23-Pin_28-Pad28)
- J23 pad 29: (no net) -> unconnected-(J23-Pin_29-Pad29)
- J23 pad 3: (no net) -> unconnected-(J23-Pin_3-Pad3)
- J23 pad 30: (no net) -> unconnected-(J23-Pin_30-Pad30)
- J23 pad 31: (no net) -> unconnected-(J23-Pin_31-Pad31)
- J23 pad 32: (no net) -> unconnected-(J23-Pin_32-Pad32)
- J23 pad 33: (no net) -> unconnected-(J23-Pin_33-Pad33)
- J23 pad 34: (no net) -> unconnected-(J23-Pin_34-Pad34)
- J23 pad 35: (no net) -> unconnected-(J23-Pin_35-Pad35)
- J23 pad 36: (no net) -> unconnected-(J23-Pin_36-Pad36)
- J23 pad 37: (no net) -> unconnected-(J23-Pin_37-Pad37)
- J23 pad 4: (no net) -> unconnected-(J23-Pin_4-Pad4)
- J23 pad 5: (no net) -> unconnected-(J23-Pin_5-Pad5)
- J23 pad 6: (no net) -> unconnected-(J23-Pin_6-Pad6)
- J23 pad 7: (no net) -> unconnected-(J23-Pin_7-Pad7)
- J23 pad 8: (no net) -> unconnected-(J23-Pin_8-Pad8)
- J23 pad 9: (no net) -> unconnected-(J23-Pin_9-Pad9)
- J24 pad 10: (no net) -> unconnected-(J24-Pin_10-Pad10)
- J24 pad 11: (no net) -> unconnected-(J24-Pin_11-Pad11)
- J24 pad 12: (no net) -> unconnected-(J24-Pin_12-Pad12)
- J24 pad 13: (no net) -> unconnected-(J24-Pin_13-Pad13)
- J24 pad 14: (no net) -> unconnected-(J24-Pin_14-Pad14)
- J24 pad 15: (no net) -> unconnected-(J24-Pin_15-Pad15)
- J24 pad 16: (no net) -> unconnected-(J24-Pin_16-Pad16)
- J24 pad 17: (no net) -> unconnected-(J24-Pin_17-Pad17)
- J24 pad 18: (no net) -> unconnected-(J24-Pin_18-Pad18)
- J24 pad 19: (no net) -> unconnected-(J24-Pin_19-Pad19)
- J24 pad 20: (no net) -> unconnected-(J24-Pin_20-Pad20)
- J24 pad 21: (no net) -> unconnected-(J24-Pin_21-Pad21)
- J24 pad 22: (no net) -> unconnected-(J24-Pin_22-Pad22)
- J24 pad 23: (no net) -> unconnected-(J24-Pin_23-Pad23)
- J24 pad 24: (no net) -> unconnected-(J24-Pin_24-Pad24)
- J24 pad 25: (no net) -> unconnected-(J24-Pin_25-Pad25)
- J24 pad 26: (no net) -> unconnected-(J24-Pin_26-Pad26)
- J24 pad 27: (no net) -> unconnected-(J24-Pin_27-Pad27)
- J24 pad 28: (no net) -> unconnected-(J24-Pin_28-Pad28)
- J24 pad 29: (no net) -> unconnected-(J24-Pin_29-Pad29)
- J24 pad 3: (no net) -> unconnected-(J24-Pin_3-Pad3)
- J24 pad 30: (no net) -> unconnected-(J24-Pin_30-Pad30)
- J24 pad 31: (no net) -> unconnected-(J24-Pin_31-Pad31)
- J24 pad 32: (no net) -> unconnected-(J24-Pin_32-Pad32)
- J24 pad 33: (no net) -> unconnected-(J24-Pin_33-Pad33)
- J24 pad 34: (no net) -> unconnected-(J24-Pin_34-Pad34)
- J24 pad 35: (no net) -> unconnected-(J24-Pin_35-Pad35)
- J24 pad 36: (no net) -> unconnected-(J24-Pin_36-Pad36)
- J24 pad 37: (no net) -> unconnected-(J24-Pin_37-Pad37)
- J24 pad 4: (no net) -> unconnected-(J24-Pin_4-Pad4)
- J24 pad 5: (no net) -> unconnected-(J24-Pin_5-Pad5)
- J24 pad 6: (no net) -> unconnected-(J24-Pin_6-Pad6)
- J24 pad 7: (no net) -> unconnected-(J24-Pin_7-Pad7)
- J24 pad 8: (no net) -> unconnected-(J24-Pin_8-Pad8)
- J24 pad 9: (no net) -> unconnected-(J24-Pin_9-Pad9)
- J25 pad 10: (no net) -> unconnected-(J25-Pin_10-Pad10)
- J25 pad 11: (no net) -> unconnected-(J25-Pin_11-Pad11)
- J25 pad 12: (no net) -> unconnected-(J25-Pin_12-Pad12)
- J25 pad 13: (no net) -> unconnected-(J25-Pin_13-Pad13)
- J25 pad 14: (no net) -> unconnected-(J25-Pin_14-Pad14)
- J25 pad 15: (no net) -> unconnected-(J25-Pin_15-Pad15)
- J25 pad 16: (no net) -> unconnected-(J25-Pin_16-Pad16)
- J25 pad 17: (no net) -> unconnected-(J25-Pin_17-Pad17)
- J25 pad 18: (no net) -> unconnected-(J25-Pin_18-Pad18)
- J25 pad 19: (no net) -> unconnected-(J25-Pin_19-Pad19)
- J25 pad 20: (no net) -> unconnected-(J25-Pin_20-Pad20)
- J25 pad 21: (no net) -> unconnected-(J25-Pin_21-Pad21)
- J25 pad 22: (no net) -> unconnected-(J25-Pin_22-Pad22)
- J25 pad 23: (no net) -> unconnected-(J25-Pin_23-Pad23)
- J25 pad 24: (no net) -> unconnected-(J25-Pin_24-Pad24)
- J25 pad 25: (no net) -> unconnected-(J25-Pin_25-Pad25)
- J25 pad 26: (no net) -> unconnected-(J25-Pin_26-Pad26)
- J25 pad 27: (no net) -> unconnected-(J25-Pin_27-Pad27)
- J25 pad 28: (no net) -> unconnected-(J25-Pin_28-Pad28)
- J25 pad 29: (no net) -> unconnected-(J25-Pin_29-Pad29)
- J25 pad 3: (no net) -> unconnected-(J25-Pin_3-Pad3)
- J25 pad 30: (no net) -> unconnected-(J25-Pin_30-Pad30)
- J25 pad 31: (no net) -> unconnected-(J25-Pin_31-Pad31)
- J25 pad 32: (no net) -> unconnected-(J25-Pin_32-Pad32)
- J25 pad 33: (no net) -> unconnected-(J25-Pin_33-Pad33)
- J25 pad 34: (no net) -> unconnected-(J25-Pin_34-Pad34)
- J25 pad 35: (no net) -> unconnected-(J25-Pin_35-Pad35)
- J25 pad 36: (no net) -> unconnected-(J25-Pin_36-Pad36)
- J25 pad 37: (no net) -> unconnected-(J25-Pin_37-Pad37)
- J25 pad 4: (no net) -> unconnected-(J25-Pin_4-Pad4)
- J25 pad 5: (no net) -> unconnected-(J25-Pin_5-Pad5)
- J25 pad 6: (no net) -> unconnected-(J25-Pin_6-Pad6)
- J25 pad 7: (no net) -> unconnected-(J25-Pin_7-Pad7)
- J25 pad 8: (no net) -> unconnected-(J25-Pin_8-Pad8)
- J25 pad 9: (no net) -> unconnected-(J25-Pin_9-Pad9)
- J26 pad 10: (no net) -> unconnected-(J26-Pin_10-Pad10)
- J26 pad 11: (no net) -> unconnected-(J26-Pin_11-Pad11)
- J26 pad 12: (no net) -> unconnected-(J26-Pin_12-Pad12)
- J26 pad 13: (no net) -> unconnected-(J26-Pin_13-Pad13)
- J26 pad 14: (no net) -> unconnected-(J26-Pin_14-Pad14)
- J26 pad 15: (no net) -> unconnected-(J26-Pin_15-Pad15)
- J26 pad 16: (no net) -> unconnected-(J26-Pin_16-Pad16)
- J26 pad 17: (no net) -> unconnected-(J26-Pin_17-Pad17)
- J26 pad 18: (no net) -> unconnected-(J26-Pin_18-Pad18)
- J26 pad 19: (no net) -> unconnected-(J26-Pin_19-Pad19)
- J26 pad 20: (no net) -> unconnected-(J26-Pin_20-Pad20)
- J26 pad 21: (no net) -> unconnected-(J26-Pin_21-Pad21)
- J26 pad 22: (no net) -> unconnected-(J26-Pin_22-Pad22)
- J26 pad 23: (no net) -> unconnected-(J26-Pin_23-Pad23)
- J26 pad 24: (no net) -> unconnected-(J26-Pin_24-Pad24)
- J26 pad 25: (no net) -> unconnected-(J26-Pin_25-Pad25)
- J26 pad 26: (no net) -> unconnected-(J26-Pin_26-Pad26)
- J26 pad 27: (no net) -> unconnected-(J26-Pin_27-Pad27)
- J26 pad 28: (no net) -> unconnected-(J26-Pin_28-Pad28)
- J26 pad 29: (no net) -> unconnected-(J26-Pin_29-Pad29)
- J26 pad 3: (no net) -> unconnected-(J26-Pin_3-Pad3)
- J26 pad 30: (no net) -> unconnected-(J26-Pin_30-Pad30)
- J26 pad 31: (no net) -> unconnected-(J26-Pin_31-Pad31)
- J26 pad 32: (no net) -> unconnected-(J26-Pin_32-Pad32)
- J26 pad 33: (no net) -> unconnected-(J26-Pin_33-Pad33)
- J26 pad 34: (no net) -> unconnected-(J26-Pin_34-Pad34)
- J26 pad 35: (no net) -> unconnected-(J26-Pin_35-Pad35)
- J26 pad 36: (no net) -> unconnected-(J26-Pin_36-Pad36)
- J26 pad 37: (no net) -> unconnected-(J26-Pin_37-Pad37)
- J26 pad 4: (no net) -> unconnected-(J26-Pin_4-Pad4)
- J26 pad 5: (no net) -> unconnected-(J26-Pin_5-Pad5)
- J26 pad 6: (no net) -> unconnected-(J26-Pin_6-Pad6)
- J26 pad 7: (no net) -> unconnected-(J26-Pin_7-Pad7)
- J26 pad 8: (no net) -> unconnected-(J26-Pin_8-Pad8)
- J26 pad 9: (no net) -> unconnected-(J26-Pin_9-Pad9)
- J27 pad 10: (no net) -> unconnected-(J27-Pin_10-Pad10)
- J27 pad 11: (no net) -> unconnected-(J27-Pin_11-Pad11)
- J27 pad 12: (no net) -> unconnected-(J27-Pin_12-Pad12)
- J27 pad 13: (no net) -> unconnected-(J27-Pin_13-Pad13)
- J27 pad 14: (no net) -> unconnected-(J27-Pin_14-Pad14)
- J27 pad 15: (no net) -> unconnected-(J27-Pin_15-Pad15)
- J27 pad 16: (no net) -> unconnected-(J27-Pin_16-Pad16)
- J27 pad 17: (no net) -> unconnected-(J27-Pin_17-Pad17)
- J27 pad 18: (no net) -> unconnected-(J27-Pin_18-Pad18)
- J27 pad 19: (no net) -> unconnected-(J27-Pin_19-Pad19)
- J27 pad 20: (no net) -> unconnected-(J27-Pin_20-Pad20)
- J27 pad 21: (no net) -> unconnected-(J27-Pin_21-Pad21)
- J27 pad 22: (no net) -> unconnected-(J27-Pin_22-Pad22)
- J27 pad 23: (no net) -> unconnected-(J27-Pin_23-Pad23)
- J27 pad 24: (no net) -> unconnected-(J27-Pin_24-Pad24)
- J27 pad 25: (no net) -> unconnected-(J27-Pin_25-Pad25)
- J27 pad 26: (no net) -> unconnected-(J27-Pin_26-Pad26)
- J27 pad 27: (no net) -> unconnected-(J27-Pin_27-Pad27)
- J27 pad 28: (no net) -> unconnected-(J27-Pin_28-Pad28)
- J27 pad 29: (no net) -> unconnected-(J27-Pin_29-Pad29)
- J27 pad 3: (no net) -> unconnected-(J27-Pin_3-Pad3)
- J27 pad 30: (no net) -> unconnected-(J27-Pin_30-Pad30)
- J27 pad 31: (no net) -> unconnected-(J27-Pin_31-Pad31)
- J27 pad 32: (no net) -> unconnected-(J27-Pin_32-Pad32)
- J27 pad 33: (no net) -> unconnected-(J27-Pin_33-Pad33)
- J27 pad 34: (no net) -> unconnected-(J27-Pin_34-Pad34)
- J27 pad 35: (no net) -> unconnected-(J27-Pin_35-Pad35)
- J27 pad 36: (no net) -> unconnected-(J27-Pin_36-Pad36)
- J27 pad 37: (no net) -> unconnected-(J27-Pin_37-Pad37)
- J27 pad 4: (no net) -> unconnected-(J27-Pin_4-Pad4)
- J27 pad 5: (no net) -> unconnected-(J27-Pin_5-Pad5)
- J27 pad 6: (no net) -> unconnected-(J27-Pin_6-Pad6)
- J27 pad 7: (no net) -> unconnected-(J27-Pin_7-Pad7)
- J27 pad 8: (no net) -> unconnected-(J27-Pin_8-Pad8)
- J27 pad 9: (no net) -> unconnected-(J27-Pin_9-Pad9)
- J28 pad 10: (no net) -> unconnected-(J28-Pin_10-Pad10)
- J28 pad 11: (no net) -> unconnected-(J28-Pin_11-Pad11)
- J28 pad 12: (no net) -> unconnected-(J28-Pin_12-Pad12)
- J28 pad 13: (no net) -> unconnected-(J28-Pin_13-Pad13)
- J28 pad 14: (no net) -> unconnected-(J28-Pin_14-Pad14)
- J28 pad 15: (no net) -> unconnected-(J28-Pin_15-Pad15)
- J28 pad 16: (no net) -> unconnected-(J28-Pin_16-Pad16)
- J28 pad 17: (no net) -> unconnected-(J28-Pin_17-Pad17)
- J28 pad 18: (no net) -> unconnected-(J28-Pin_18-Pad18)
- J28 pad 19: (no net) -> unconnected-(J28-Pin_19-Pad19)
- J28 pad 20: (no net) -> unconnected-(J28-Pin_20-Pad20)
- J28 pad 21: (no net) -> unconnected-(J28-Pin_21-Pad21)
- J28 pad 22: (no net) -> unconnected-(J28-Pin_22-Pad22)
- J28 pad 23: (no net) -> unconnected-(J28-Pin_23-Pad23)
- J28 pad 24: (no net) -> unconnected-(J28-Pin_24-Pad24)
- J28 pad 25: (no net) -> unconnected-(J28-Pin_25-Pad25)
- J28 pad 26: (no net) -> unconnected-(J28-Pin_26-Pad26)
- J28 pad 27: (no net) -> unconnected-(J28-Pin_27-Pad27)
- J28 pad 28: (no net) -> unconnected-(J28-Pin_28-Pad28)
- J28 pad 29: (no net) -> unconnected-(J28-Pin_29-Pad29)
- J28 pad 3: (no net) -> unconnected-(J28-Pin_3-Pad3)
- J28 pad 30: (no net) -> unconnected-(J28-Pin_30-Pad30)
- J28 pad 31: (no net) -> unconnected-(J28-Pin_31-Pad31)
- J28 pad 32: (no net) -> unconnected-(J28-Pin_32-Pad32)
- J28 pad 33: (no net) -> unconnected-(J28-Pin_33-Pad33)
- J28 pad 34: (no net) -> unconnected-(J28-Pin_34-Pad34)
- J28 pad 35: (no net) -> unconnected-(J28-Pin_35-Pad35)
- J28 pad 36: (no net) -> unconnected-(J28-Pin_36-Pad36)
- J28 pad 37: (no net) -> unconnected-(J28-Pin_37-Pad37)
- J28 pad 4: (no net) -> unconnected-(J28-Pin_4-Pad4)
- J28 pad 5: (no net) -> unconnected-(J28-Pin_5-Pad5)
- J28 pad 6: (no net) -> unconnected-(J28-Pin_6-Pad6)
- J28 pad 7: (no net) -> unconnected-(J28-Pin_7-Pad7)
- J28 pad 8: (no net) -> unconnected-(J28-Pin_8-Pad8)
- J28 pad 9: (no net) -> unconnected-(J28-Pin_9-Pad9)
- J29 pad 10: (no net) -> unconnected-(J29-Pin_10-Pad10)
- J29 pad 11: (no net) -> unconnected-(J29-Pin_11-Pad11)
- J29 pad 12: (no net) -> unconnected-(J29-Pin_12-Pad12)
- J29 pad 13: (no net) -> unconnected-(J29-Pin_13-Pad13)
- J29 pad 14: (no net) -> unconnected-(J29-Pin_14-Pad14)
- J29 pad 15: (no net) -> unconnected-(J29-Pin_15-Pad15)
- J29 pad 16: (no net) -> unconnected-(J29-Pin_16-Pad16)
- J29 pad 17: (no net) -> unconnected-(J29-Pin_17-Pad17)
- J29 pad 18: (no net) -> unconnected-(J29-Pin_18-Pad18)
- J29 pad 19: (no net) -> unconnected-(J29-Pin_19-Pad19)
- J29 pad 20: (no net) -> unconnected-(J29-Pin_20-Pad20)
- J29 pad 21: (no net) -> unconnected-(J29-Pin_21-Pad21)
- J29 pad 22: (no net) -> unconnected-(J29-Pin_22-Pad22)
- J29 pad 23: (no net) -> unconnected-(J29-Pin_23-Pad23)
- J29 pad 24: (no net) -> unconnected-(J29-Pin_24-Pad24)
- J29 pad 25: (no net) -> unconnected-(J29-Pin_25-Pad25)
- J29 pad 26: (no net) -> unconnected-(J29-Pin_26-Pad26)
- J29 pad 27: (no net) -> unconnected-(J29-Pin_27-Pad27)
- J29 pad 28: (no net) -> unconnected-(J29-Pin_28-Pad28)
- J29 pad 29: (no net) -> unconnected-(J29-Pin_29-Pad29)
- J29 pad 3: (no net) -> unconnected-(J29-Pin_3-Pad3)
- J29 pad 30: (no net) -> unconnected-(J29-Pin_30-Pad30)
- J29 pad 31: (no net) -> unconnected-(J29-Pin_31-Pad31)
- J29 pad 32: (no net) -> unconnected-(J29-Pin_32-Pad32)
- J29 pad 33: (no net) -> unconnected-(J29-Pin_33-Pad33)
- J29 pad 34: (no net) -> unconnected-(J29-Pin_34-Pad34)
- J29 pad 35: (no net) -> unconnected-(J29-Pin_35-Pad35)
- J29 pad 36: (no net) -> unconnected-(J29-Pin_36-Pad36)
- J29 pad 37: (no net) -> unconnected-(J29-Pin_37-Pad37)
- J29 pad 4: (no net) -> unconnected-(J29-Pin_4-Pad4)
- J29 pad 5: (no net) -> unconnected-(J29-Pin_5-Pad5)
- J29 pad 6: (no net) -> unconnected-(J29-Pin_6-Pad6)
- J29 pad 7: (no net) -> unconnected-(J29-Pin_7-Pad7)
- J29 pad 8: (no net) -> unconnected-(J29-Pin_8-Pad8)
- J29 pad 9: (no net) -> unconnected-(J29-Pin_9-Pad9)
- J30 pad 10: (no net) -> unconnected-(J30-Pin_10-Pad10)
- J30 pad 11: (no net) -> unconnected-(J30-Pin_11-Pad11)
- J30 pad 12: (no net) -> unconnected-(J30-Pin_12-Pad12)
- J30 pad 13: (no net) -> unconnected-(J30-Pin_13-Pad13)
- J30 pad 14: (no net) -> unconnected-(J30-Pin_14-Pad14)
- J30 pad 15: (no net) -> unconnected-(J30-Pin_15-Pad15)
- J30 pad 16: (no net) -> unconnected-(J30-Pin_16-Pad16)
- J30 pad 17: (no net) -> unconnected-(J30-Pin_17-Pad17)
- J30 pad 18: (no net) -> unconnected-(J30-Pin_18-Pad18)
- J30 pad 19: (no net) -> unconnected-(J30-Pin_19-Pad19)
- J30 pad 20: (no net) -> unconnected-(J30-Pin_20-Pad20)
- J30 pad 21: (no net) -> unconnected-(J30-Pin_21-Pad21)
- J30 pad 22: (no net) -> unconnected-(J30-Pin_22-Pad22)
- J30 pad 23: (no net) -> unconnected-(J30-Pin_23-Pad23)
- J30 pad 24: (no net) -> unconnected-(J30-Pin_24-Pad24)
- J30 pad 25: (no net) -> unconnected-(J30-Pin_25-Pad25)
- J30 pad 26: (no net) -> unconnected-(J30-Pin_26-Pad26)
- J30 pad 27: (no net) -> unconnected-(J30-Pin_27-Pad27)
- J30 pad 28: (no net) -> unconnected-(J30-Pin_28-Pad28)
- J30 pad 29: (no net) -> unconnected-(J30-Pin_29-Pad29)
- J30 pad 3: (no net) -> unconnected-(J30-Pin_3-Pad3)
- J30 pad 30: (no net) -> unconnected-(J30-Pin_30-Pad30)
- J30 pad 31: (no net) -> unconnected-(J30-Pin_31-Pad31)
- J30 pad 32: (no net) -> unconnected-(J30-Pin_32-Pad32)
- J30 pad 33: (no net) -> unconnected-(J30-Pin_33-Pad33)
- J30 pad 34: (no net) -> unconnected-(J30-Pin_34-Pad34)
- J30 pad 35: (no net) -> unconnected-(J30-Pin_35-Pad35)
- J30 pad 36: (no net) -> unconnected-(J30-Pin_36-Pad36)
- J30 pad 37: (no net) -> unconnected-(J30-Pin_37-Pad37)
- J30 pad 4: (no net) -> unconnected-(J30-Pin_4-Pad4)
- J30 pad 5: (no net) -> unconnected-(J30-Pin_5-Pad5)
- J30 pad 6: (no net) -> unconnected-(J30-Pin_6-Pad6)
- J30 pad 7: (no net) -> unconnected-(J30-Pin_7-Pad7)
- J30 pad 8: (no net) -> unconnected-(J30-Pin_8-Pad8)
- J30 pad 9: (no net) -> unconnected-(J30-Pin_9-Pad9)
- J31 pad 10: (no net) -> unconnected-(J31-Pin_10-Pad10)
- J31 pad 11: (no net) -> unconnected-(J31-Pin_11-Pad11)
- J31 pad 12: (no net) -> unconnected-(J31-Pin_12-Pad12)
- J31 pad 13: (no net) -> unconnected-(J31-Pin_13-Pad13)
- J31 pad 14: (no net) -> unconnected-(J31-Pin_14-Pad14)
- J31 pad 15: (no net) -> unconnected-(J31-Pin_15-Pad15)
- J31 pad 16: (no net) -> unconnected-(J31-Pin_16-Pad16)
- J31 pad 17: (no net) -> unconnected-(J31-Pin_17-Pad17)
- J31 pad 18: (no net) -> unconnected-(J31-Pin_18-Pad18)
- J31 pad 19: (no net) -> unconnected-(J31-Pin_19-Pad19)
- J31 pad 20: (no net) -> unconnected-(J31-Pin_20-Pad20)
- J31 pad 21: (no net) -> unconnected-(J31-Pin_21-Pad21)
- J31 pad 22: (no net) -> unconnected-(J31-Pin_22-Pad22)
- J31 pad 23: (no net) -> unconnected-(J31-Pin_23-Pad23)
- J31 pad 24: (no net) -> unconnected-(J31-Pin_24-Pad24)
- J31 pad 25: (no net) -> unconnected-(J31-Pin_25-Pad25)
- J31 pad 26: (no net) -> unconnected-(J31-Pin_26-Pad26)
- J31 pad 27: (no net) -> unconnected-(J31-Pin_27-Pad27)
- J31 pad 28: (no net) -> unconnected-(J31-Pin_28-Pad28)
- J31 pad 29: (no net) -> unconnected-(J31-Pin_29-Pad29)
- J31 pad 3: (no net) -> unconnected-(J31-Pin_3-Pad3)
- J31 pad 30: (no net) -> unconnected-(J31-Pin_30-Pad30)
- J31 pad 31: (no net) -> unconnected-(J31-Pin_31-Pad31)
- J31 pad 32: (no net) -> unconnected-(J31-Pin_32-Pad32)
- J31 pad 33: (no net) -> unconnected-(J31-Pin_33-Pad33)
- J31 pad 34: (no net) -> unconnected-(J31-Pin_34-Pad34)
- J31 pad 35: (no net) -> unconnected-(J31-Pin_35-Pad35)
- J31 pad 36: (no net) -> unconnected-(J31-Pin_36-Pad36)
- J31 pad 37: (no net) -> unconnected-(J31-Pin_37-Pad37)
- J31 pad 4: (no net) -> unconnected-(J31-Pin_4-Pad4)
- J31 pad 5: (no net) -> unconnected-(J31-Pin_5-Pad5)
- J31 pad 6: (no net) -> unconnected-(J31-Pin_6-Pad6)
- J31 pad 7: (no net) -> unconnected-(J31-Pin_7-Pad7)
- J31 pad 8: (no net) -> unconnected-(J31-Pin_8-Pad8)
- J31 pad 9: (no net) -> unconnected-(J31-Pin_9-Pad9)
- J32 pad 10: (no net) -> unconnected-(J32-Pin_10-Pad10)
- J32 pad 11: (no net) -> unconnected-(J32-Pin_11-Pad11)
- J32 pad 12: (no net) -> unconnected-(J32-Pin_12-Pad12)
- J32 pad 13: (no net) -> unconnected-(J32-Pin_13-Pad13)
- J32 pad 14: (no net) -> unconnected-(J32-Pin_14-Pad14)
- J32 pad 15: (no net) -> unconnected-(J32-Pin_15-Pad15)
- J32 pad 16: (no net) -> unconnected-(J32-Pin_16-Pad16)
- J32 pad 17: (no net) -> unconnected-(J32-Pin_17-Pad17)
- J32 pad 18: (no net) -> unconnected-(J32-Pin_18-Pad18)
- J32 pad 19: (no net) -> unconnected-(J32-Pin_19-Pad19)
- J32 pad 2: (no net) -> unconnected-(J32-Pin_2-Pad2)
- J32 pad 20: (no net) -> unconnected-(J32-Pin_20-Pad20)
- J32 pad 21: (no net) -> unconnected-(J32-Pin_21-Pad21)
- J32 pad 22: (no net) -> unconnected-(J32-Pin_22-Pad22)
- J32 pad 23: (no net) -> unconnected-(J32-Pin_23-Pad23)
- J32 pad 24: (no net) -> unconnected-(J32-Pin_24-Pad24)
- J32 pad 25: (no net) -> unconnected-(J32-Pin_25-Pad25)
- J32 pad 26: (no net) -> unconnected-(J32-Pin_26-Pad26)
- J32 pad 27: (no net) -> unconnected-(J32-Pin_27-Pad27)
- J32 pad 28: (no net) -> unconnected-(J32-Pin_28-Pad28)
- J32 pad 29: (no net) -> unconnected-(J32-Pin_29-Pad29)
- J32 pad 3: (no net) -> unconnected-(J32-Pin_3-Pad3)
- J32 pad 30: (no net) -> unconnected-(J32-Pin_30-Pad30)
- J32 pad 31: (no net) -> unconnected-(J32-Pin_31-Pad31)
- J32 pad 4: (no net) -> unconnected-(J32-Pin_4-Pad4)
- J32 pad 5: (no net) -> unconnected-(J32-Pin_5-Pad5)
- J32 pad 6: (no net) -> unconnected-(J32-Pin_6-Pad6)
- J32 pad 7: (no net) -> unconnected-(J32-Pin_7-Pad7)
- J32 pad 8: (no net) -> unconnected-(J32-Pin_8-Pad8)
- J32 pad 9: (no net) -> unconnected-(J32-Pin_9-Pad9)
Routing:
- net /RX2: track 45.6 -> 46.7 mm
