File: Fill_Memory_Board/bus.kicad_sch (KiCad schematic)
At the start: 4 parts

Commit message: Readme update
Changed lines of the file:
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@@
     (effects (font (size 1.27 1.27)) (justify left))
   )
-  (hierarchical_label "TX3" (shape input) (at 123.825 96.52 180) (fields_autoplaced)
+  (hierarchical_label "TX3" (shape output) (at 123.825 96.52 180) (fields_autoplaced)
     (effects (font (size 1.27 1.27)) (justify right))
   )
