File: MultiParallel v2/schematic/MOS_MultiParallel_2/MOS_MultiParallel_2.kicad_pcb (KiCad board)
At the start: 2 copper layers, 100 x 100 mm, 64 parts, among them J1 BUS, J10 ., J11 ., J12 Conn_01x01, J13 ., J14 ., J15 ., J16 ., J17 Conn_01x01, J18 Conn_01x01, J2 BUS, J20 Conn_01x12, J21 Conn_01x12, J25 ., J26 .Conn_01x01, J27 ., J28 ., J29 ., J3 BUS, J30 ., J31 Conn_02x22_Odd_Even, J4 BUS, J5 ., J6 ., J7 ., J8 ., J9 Conn_01x01, U1 SN74LVCC4245ANSR, U11 W65C22NxP, U2 74HC14, U3 6532, U4 W65C22NxP, U5 IS63WV1288DBLL-10xLI, U6 74LVC253, U7 74LVC595, U8 74AHC1G14

Commit message: Readme update
Connections:
- J2 pad 3: /RX2 -> /TX2
- J2 pad 4: /TX2 -> /RX2
- J2 pad 5: /RX3 -> /TX3
- J2 pad 6: /TX3 -> /RX3
- J4 pad 3: /RX2 -> /TX2
- J4 pad 4: /TX2 -> /RX2
- J4 pad 5: /RX3 -> /TX3
- J4 pad 6: /TX3 -> /RX3
Changed lines of the file:
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@@
       (net 16 "+5V") (pinfunction "Pin_2") (pintype "passive"))
     (pad "3" thru_hole oval (at 0 2.54 90) (size 1.7 1.7) (drill 1) (layers "*.Cu" "*.Mask")
-      (net 68 "/RX2") (pinfunction "Pin_3") (pintype "passive"))
+      (net 67 "/TX2") (pinfunction "Pin_3") (pintype "passive"))
     (pad "4" thru_hole oval (at -2.54 2.54 90) (size 1.7 1.7) (drill 1) (layers "*.Cu" "*.Mask")
-      (net 67 "/TX2") (pinfunction "Pin_4") (pintype "passive"))
+      (net 68 "/RX2") (pinfunction "Pin_4") (pintype "passive"))
     (pad "5" thru_hole oval (at 0 5.08 90) (size 1.7 1.7) (drill 1) (layers "*.Cu" "*.Mask")
-      (net 66 "/RX3") (pinfunction "Pin_5") (pintype "passive"))
+      (net 65 "/TX3") (pinfunction "Pin_5") (pintype "passive"))
     (pad "6" thru_hole oval (at -2.54 5.08 90) (size 1.7 1.7) (drill 1) (layers "*.Cu" "*.Mask")
-      (net 65 "/TX3") (pinfunction "Pin_6") (pintype "passive"))
+      (net 66 "/RX3") (pinfunction "Pin_6") (pintype "passive"))
     (pad "7" thru_hole oval (at 0 7.62 90) (size 1.7 1.7) (drill 1) (layers "*.Cu" "*.Mask")
       (net 64 "/RES0") (pinfunction "Pin_7") (pintype "passive"))
@@
       (net 16 "+5V") (pinfunction "Pin_2") (pintype "passive"))
     (pad "3" thru_hole oval (at 0 2.54 90) (size 1.7 1.7) (drill 1) (layers "*.Cu" "*.Mask")
-      (net 68 "/RX2") (pinfunction "Pin_3") (pintype "passive"))
+      (net 67 "/TX2") (pinfunction "Pin_3") (pintype "passive"))
     (pad "4" thru_hole oval (at -2.54 2.54 90) (size 1.7 1.7) (drill 1) (layers "*.Cu" "*.Mask")
-      (net 67 "/TX2") (pinfunction "Pin_4") (pintype "passive"))
+      (net 68 "/RX2") (pinfunction "Pin_4") (pintype "passive"))
     (pad "5" thru_hole oval (at 0 5.08 90) (size 1.7 1.7) (drill 1) (layers "*.Cu" "*.Mask")
-      (net 66 "/RX3") (pinfunction "Pin_5") (pintype "passive"))
+      (net 65 "/TX3") (pinfunction "Pin_5") (pintype "passive"))
     (pad "6" thru_hole oval (at -2.54 5.08 90) (size 1.7 1.7) (drill 1) (layers "*.Cu" "*.Mask")
-      (net 65 "/TX3") (pinfunction "Pin_6") (pintype "passive"))
+      (net 66 "/RX3") (pinfunction "Pin_6") (pintype "passive"))
     (pad "7" thru_hole oval (at 0 7.62 90) (size 1.7 1.7) (drill 1) (layers "*.Cu" "*.Mask")
       (net 64 "/RES0") (pinfunction "Pin_7") (pintype "passive"))
@@
   (segment (start 146.07 135.099005) (end 147.32 133.849005) (width 0.4) (layer "B.Cu") (net 64))
   (segment (start 147.32 139.7) (end 147.32 138.497919) (width 0.4) (layer "B.Cu") (net 64))
-  (segment (start 144.78 136.017) (end 144.78 137.287) (width 0.4) (layer "B.Cu") (net 65))
-  (segment (start 146.05 138.557) (end 146.05 140.97) (width 0.4) (layer "B.Cu") (net 65))
-  (segment (start 146.05 140.97) (end 144.78 142.24) (width 0.4) (layer "B.Cu") (net 65))
-  (segment (start 144.78 137.287) (end 146.05 138.557) (width 0.4) (layer "B.Cu") (net 65))
-  (segment (start 144.78 134.621238) (end 144.78 133.849005) (width 0.4) (layer "B.Cu") (net 66))
-  (segment (start 143.53 137.18) (end 143.53 135.871238) (width 0.4) (layer "B.Cu") (net 66))
-  (segment (start 143.53 135.871238) (end 144.78 134.621238) (width 0.4) (layer "B.Cu") (net 66))
-  (segment (start 144.78 138.43) (end 143.53 137.18) (width 0.4) (layer "B.Cu") (net 66))
-  (segment (start 144.78 139.623705) (end 144.78 138.43) (width 0.4) (layer "B.Cu") (net 66))
-  (segment (start 143.49 140.99) (end 142.24 142.24) (width 0.4) (layer "B.Cu") (net 67))
-  (segment (start 143.49 138.537) (end 143.49 140.99) (width 0.4) (layer "B.Cu") (net 67))
-  (segment (start 142.24 136.017) (end 142.24 137.287) (width 0.4) (layer "B.Cu") (net 67))
-  (segment (start 142.24 137.287) (end 143.49 138.537) (width 0.4) (layer "B.Cu") (net 67))
-  (segment (start 140.99 138.45) (end 140.99 135.099005) (width 0.4) (layer "B.Cu") (net 68))
-  (segment (start 140.99 135.099005) (end 142.24 133.849005) (width 0.4) (layer "B.Cu") (net 68))
-  (segment (start 142.24 139.7) (end 140.99 138.45) (width 0.4) (layer "B.Cu") (net 68))
+  (segment (start 144.78 134.621238) (end 144.78 133.849005) (width 0.4) (layer "B.Cu") (net 65))
+  (segment (start 143.53 137.18) (end 143.53 135.871238) (width 0.4) (layer "B.Cu") (net 65))
+  (segment (start 143.53 135.871238) (end 144.78 134.621238) (width 0.4) (layer "B.Cu") (net 65))
+  (segment (start 144.78 138.43) (end 143.53 137.18) (width 0.4) (layer "B.Cu") (net 65))
+  (segment (start 144.78 139.623705) (end 144.78 138.43) (width 0.4) (layer "B.Cu") (net 65))
+  (segment (start 144.78 136.017) (end 144.78 137.287) (width 0.4) (layer "B.Cu") (net 66))
+  (segment (start 146.05 138.557) (end 146.05 140.97) (width 0.4) (layer "B.Cu") (net 66))
+  (segment (start 146.05 140.97) (end 144.78 142.24) (width 0.4) (layer "B.Cu") (net 66))
+  (segment (start 144.78 137.287) (end 146.05 138.557) (width 0.4) (layer "B.Cu") (net 66))
+  (segment (start 140.99 138.45) (end 140.99 135.099005) (width 0.4) (layer "B.Cu") (net 67))
+  (segment (start 140.99 135.099005) (end 142.24 133.849005) (width 0.4) (layer "B.Cu") (net 67))
+  (segment (start 142.24 139.7) (end 140.99 138.45) (width 0.4) (layer "B.Cu") (net 67))
+  (segment (start 143.49 140.99) (end 142.24 142.24) (width 0.4) (layer "B.Cu") (net 68))
+  (segment (start 143.49 138.537) (end 143.49 140.99) (width 0.4) (layer "B.Cu") (net 68))
+  (segment (start 142.24 136.017) (end 142.24 137.287) (width 0.4) (layer "B.Cu") (net 68))
+  (segment (start 142.24 137.287) (end 143.49 138.537) (width 0.4) (layer "B.Cu") (net 68))
   (segment (start 177.8 136.779) (end 179.05 138.029) (width 0.4) (layer "B.Cu") (net 69))
   (segment (start 179.05 138.029) (end 179.05 140.99) (width 0.4) (layer "B.Cu") (net 69))
