File: MultiParallel v2/schematic/MOS_MultiParallel_2/bus.kicad_sch (KiCad schematic)
At the start: 8 parts, among them J12 Conn_01x01, U1 SN74LVCC4245ANSR

Commit message: Readme update
Connections:
- net RX2: now also J?.3 (Pin_3), J?.3 (Pin_3); no longer J?.4 (Pin_4), J?.4 (Pin_4)
- net RX3: now also J?.5 (Pin_5), J?.5 (Pin_5); no longer J?.6 (Pin_6), J?.6 (Pin_6)
- net TX2: now also J?.4 (Pin_4), J?.4 (Pin_4); no longer J?.3 (Pin_3), J?.3 (Pin_3)
- net TX3: now also J?.6 (Pin_6), J?.6 (Pin_6); no longer J?.5 (Pin_5), J?.5 (Pin_5)
Changed lines of the file:
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@@
     (effects (font (size 1.27 1.27)) (justify left bottom))
   )
-  (label "RX2" (at 102.235 93.98 180) (fields_autoplaced)
-    (effects (font (size 1.27 1.27)) (justify right bottom))
+  (label "RX2" (at 64.135 93.98 0) (fields_autoplaced)
+    (effects (font (size 1.27 1.27)) (justify left bottom))
   )
   (label "~{RAMWE9}" (at 184.15 118.11 0) (fields_autoplaced)
@@
     (effects (font (size 1.27 1.27)) (justify left bottom))
   )
-  (label "RX3" (at 102.235 96.52 180) (fields_autoplaced)
-    (effects (font (size 1.27 1.27)) (justify right bottom))
+  (label "RX3" (at 64.135 96.52 0) (fields_autoplaced)
+    (effects (font (size 1.27 1.27)) (justify left bottom))
   )
   (label "A6" (at 125.73 57.15 0) (fields_autoplaced)
@@
     (effects (font (size 1.27 1.27)) (justify right bottom))
   )
-  (label "TX3" (at 64.135 96.52 0) (fields_autoplaced)
-    (effects (font (size 1.27 1.27)) (justify left bottom))
+  (label "TX3" (at 102.235 96.52 180) (fields_autoplaced)
+    (effects (font (size 1.27 1.27)) (justify right bottom))
   )
   (label "PHI1_e" (at 63.5 29.21 0) (fields_autoplaced)
@@
     (effects (font (size 1.27 1.27)) (justify right bottom))
   )
-  (label "TX2" (at 64.135 93.98 0) (fields_autoplaced)
-    (effects (font (size 1.27 1.27)) (justify left bottom))
+  (label "TX2" (at 102.235 93.98 180) (fields_autoplaced)
+    (effects (font (size 1.27 1.27)) (justify right bottom))
   )
   (label "~{RAMWE9}" (at 161.925 114.3 180) (fields_autoplaced)
@@
     (effects (font (size 1.27 1.27)) (justify right))
   )
-  (hierarchical_label "RX2" (shape input) (at 163.195 93.98 0) (fields_autoplaced)
-    (effects (font (size 1.27 1.27)) (justify left))
+  (hierarchical_label "RX2" (shape input) (at 123.825 93.98 180) (fields_autoplaced)
+    (effects (font (size 1.27 1.27)) (justify right))
   )
   (hierarchical_label "RX_3V" (shape input) (at 163.195 101.6 0) (fields_autoplaced)
@@
     (effects (font (size 1.27 1.27)) (justify right))
   )
-  (hierarchical_label "TX3" (shape input) (at 123.825 96.52 180) (fields_autoplaced)
-    (effects (font (size 1.27 1.27)) (justify right))
+  (hierarchical_label "TX3" (shape output) (at 163.195 96.52 0) (fields_autoplaced)
+    (effects (font (size 1.27 1.27)) (justify left))
   )
   (hierarchical_label "~{DOE}" (shape input) (at 172.085 64.135 180) (fields_autoplaced)
@@
     (effects (font (size 1.27 1.27)) (justify right))
   )
-  (hierarchical_label "TX2" (shape output) (at 123.825 93.98 180) (fields_autoplaced)
-    (effects (font (size 1.27 1.27)) (justify right))
+  (hierarchical_label "TX2" (shape output) (at 163.195 93.98 0) (fields_autoplaced)
+    (effects (font (size 1.27 1.27)) (justify left))
   )
   (hierarchical_label "TDI" (shape input) (at 158.115 134.62 0) (fields_autoplaced)
@@
     (effects (font (size 1.27 1.27)) (justify left))
   )
-  (hierarchical_label "RX3" (shape input) (at 163.195 96.52 0) (fields_autoplaced)
-    (effects (font (size 1.27 1.27)) (justify left))
+  (hierarchical_label "RX3" (shape input) (at 123.825 96.52 180) (fields_autoplaced)
+    (effects (font (size 1.27 1.27)) (justify right))
   )
   (symbol (lib_id "Connector_Generic:Conn_01x01") (at 180.975 61.595 0) (mirror y) (unit 1)
