File: RAMROM_128k_board/RAMROM_128k_board.kicad_pcb (KiCad board)
At the start: 2 copper layers, 100 x 100 mm, 46 parts, among them J1 BUS, J2 BUS, J3 BUS, J4 BUS, J6 STM32F411, J7 ., J8 ., J9 ., Q1 PMV450ENEAR, U1 SN74LVC245ANSR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

Commit message: Readme update
Routing:
- net /RX2: track 40.2 -> 39.7 mm, vias 1 -> 2
- net /CNT: vias 2 -> 1
