File: RAMROM_128k_board/RAMROM_128k_board.kicad_sch (KiCad schematic)
At the start: 45 parts, among them J10 ., J11 ., J5 ., J6 STM32F411, J7 ., J8 ., J9 ., Q1 PMV450ENEAR, U1 SN74LVC245ANSR, U10 74LVC595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

Commit message: Readme update
Parts:
- removed J10, J11, J5: ., Connector_PinHeader_2.00mm:PinHeader_1x01_P2.00mm_Vertical, symbol Connector_Generic:Conn_01x01
Changed lines of the file:
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@@
     (stroke (width 0) (type default))
   )
-  (wire (pts (xy 60.325 154.94) (xy 59.69 154.94))
-    (stroke (width 0) (type default))
-  )
   (wire (pts (xy 295.275 41.91) (xy 312.42 41.91))
     (stroke (width 0) (type default))
@@
     (stroke (width 0) (type default))
   )
-  (wire (pts (xy 41.275 160.655) (xy 60.325 160.655))
-    (stroke (width 0) (type default))
-  )
   (wire (pts (xy 238.76 38.1) (xy 238.76 88.265))
     (stroke (width 0) (type default))
@@
     (stroke (width 0) (type default))
   )
-  (wire (pts (xy 60.325 160.655) (xy 60.325 154.94))
-    (stroke (width 0) (type default))
-  )
   (wire (pts (xy 242.57 33.02) (xy 242.57 83.185))
     (stroke (width 0) (type default))
@@
     (effects (font (size 1.27 1.27)) (justify left bottom))
   )
-  (label "TX2" (at 14.605 46.355 0) (fields_autoplaced)
+  (label "TX2" (at 14.605 43.815 0) (fields_autoplaced)
     (effects (font (size 1.27 1.27)) (justify left bottom))
   )
@@
     (effects (font (size 1.27 1.27)) (justify left bottom))
   )
-  (label "TX3" (at 14.605 51.435 0) (fields_autoplaced)
+  (label "TX3" (at 14.605 48.895 0) (fields_autoplaced)
     (effects (font (size 1.27 1.27)) (justify left bottom))
   )
@@
     (effects (font (size 1.27 1.27)) (justify left bottom))
   )
-  (label "RX3" (at 14.605 48.895 0) (fields_autoplaced)
+  (label "RX3" (at 14.605 51.435 0) (fields_autoplaced)
     (effects (font (size 1.27 1.27)) (justify left bottom))
   )
@@
     (effects (font (size 1.27 1.27)) (justify left bottom))
   )
-  (label "RX2" (at 14.605 43.815 0) (fields_autoplaced)
+  (label "RX2" (at 14.605 46.355 0) (fields_autoplaced)
     (effects (font (size 1.27 1.27)) (justify left bottom))
   )
@@
     )
   )
-  (symbol (lib_id "Connector_Generic:Conn_01x01") (at 36.195 160.655 0) (mirror y) (unit 1)
-    (in_bom yes) (on_board yes) (dnp no)
-    (property "Reference" "J11" (at 34.163 159.8203 0)
-      (effects (font (size 1.27 1.27)) (justify left))
-    )
-    (property "Value" "." (at 40.64 157.48 0)
-      (effects (font (size 1.27 1.27)) (justify left))
-    )
-    (property "Footprint" "Connector_PinHeader_2.00mm:PinHeader_1x01_P2.00mm_Vertical" (at 36.195 160.655 0)
-      (effects (font (size 1.27 1.27)) hide)
-    )
-    (property "Datasheet" "~" (at 36.195 160.655 0)
-      (effects (font (size 1.27 1.27)) hide)
-    )
-    (pin "1")
-    (instances
-      (project "RAMROM_128k_board"
-        (path "/2eaa3998-c9cb-43b1-9b23-df656c8158b0"
-          (reference "J11") (unit 1)
-        )
-      )
-    )
-  )
-  (symbol (lib_id "Connector_Generic:Conn_01x01") (at 39.37 157.48 0) (mirror y) (unit 1)
-    (in_bom yes) (on_board yes) (dnp no)
-    (property "Reference" "J5" (at 37.338 156.6453 0)
-      (effects (font (size 1.27 1.27)) (justify left))
-    )
-    (property "Value" "." (at 43.815 154.305 0)
-      (effects (font (size 1.27 1.27)) (justify left))
-    )
-    (property "Footprint" "Connector_PinHeader_2.00mm:PinHeader_1x01_P2.00mm_Vertical" (at 39.37 157.48 0)
-      (effects (font (size 1.27 1.27)) hide)
-    )
-    (property "Datasheet" "~" (at 39.37 157.48 0)
-      (effects (font (size 1.27 1.27)) hide)
-    )
-    (pin "1")
-    (instances
-      (project "RAMROM_128k_board"
-        (path "/2eaa3998-c9cb-43b1-9b23-df656c8158b0"
-          (reference "J5") (unit 1)
-        )
-      )
-    )
-  )
   (symbol (lib_id "power:GND") (at 322.58 152.4 0) (unit 1)
     (in_bom yes) (on_board yes) (dnp no) (fields_autoplaced)
@@
         )
       )
-    )
-  )
-  (symbol (lib_id "Connector_Generic:Conn_01x01") (at 39.37 152.4 0) (mirror y) (unit 1)
-    (in_bom yes) (on_board yes) (dnp no)
-    (property "Reference" "J10" (at 37.338 151.5653 0)
-      (effects (font (size 1.27 1.27)) (justify left))
-    )
-    (property "Value" "." (at 43.815 149.225 0)
-      (effects (font (size 1.27 1.27)) (justify left))
-    )
-    (property "Footprint" "Connector_PinHeader_2.00mm:PinHeader_1x01_P2.00mm_Vertical" (at 39.37 152.4 0)
-      (effects (font (size 1.27 1.27)) hide)
-    )
-    (property "Datasheet" "~" (at 39.37 152.4 0)
-      (effects (font (size 1.27 1.27)) hide)
-    )
-    (pin "1")
-    (instances
-      (project "RAMROM_128k_board"
-        (path "/2eaa3998-c9cb-43b1-9b23-df656c8158b0"
-          (reference "J10") (unit 1)
-        )
-      )
