File: RAMROM_Board_v3/RAMROM_Board_v3.kicad_pcb (KiCad board)
At the start: 2 copper layers, 100 x 100 mm, 41 parts, among them J1 BUS, J10 ., J11 ., J2 BUS, J20 Conn_01x12, J21 Conn_01x12, J3 BUS, J4 BUS, J8 ., U1 SN74LVC245ANSR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

Commit message: Readme update
Parts:
- added C10: 100n, Capacitor_SMD:C_1206_3216Metric, F.Cu at (86.3, 94.4)
Connections:
- J2 pad 3: /RX2 -> /TX2
- J2 pad 4: /TX2 -> /RX2
- J2 pad 5: /RX3 -> /TX3
- J2 pad 6: /TX3 -> /RX3
- J4 pad 3: /RX2 -> /TX2
- J4 pad 4: /TX2 -> /RX2
- J4 pad 5: /RX3 -> /TX3
- J4 pad 6: /TX3 -> /RX3
Changed lines of the file:
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@@
     (fp_line (start -2.45 3.25) (end 3.5 3.25)
       (stroke (width 0.05) (type solid)) (layer "F.CrtYd"))
-    (fp_arc (start 3.5 3.25) (mid 3.80926 3.345922) (end 4.01 3.6)
+    (fp_arc (start 3.5 3.25) (mid 3.809266 3.345926) (end 4.01 3.6)
       (stroke (width 0.05) (type solid)) (layer "F.CrtYd"))
     (fp_arc (start 4.01 -3.6) (mid 3.809274 -3.345915) (end 3.5 -3.25)
@@
       (net 11 "+5V") (pinfunction "Pin_2") (pintype "passive"))
     (pad "3" thru_hole oval (at 0 2.54 90) (size 1.7 1.7) (drill 1) (layers "*.Cu" "*.Mask")
-      (net 53 "/RX2") (pinfunction "Pin_3") (pintype "passive"))
+      (net 52 "/TX2") (pinfunction "Pin_3") (pintype "passive"))
     (pad "4" thru_hole oval (at -2.54 2.54 90) (size 1.7 1.7) (drill 1) (layers "*.Cu" "*.Mask")
-      (net 52 "/TX2") (pinfunction "Pin_4") (pintype "passive"))
+      (net 53 "/RX2") (pinfunction "Pin_4") (pintype "passive"))
     (pad "5" thru_hole oval (at 0 5.08 90) (size 1.7 1.7) (drill 1) (layers "*.Cu" "*.Mask")
-      (net 51 "/RX3") (pinfunction "Pin_5") (pintype "passive"))
+      (net 50 "/TX3") (pinfunction "Pin_5") (pintype "passive"))
     (pad "6" thru_hole oval (at -2.54 5.08 90) (size 1.7 1.7) (drill 1) (layers "*.Cu" "*.Mask")
-      (net 50 "/TX3") (pinfunction "Pin_6") (pintype "passive"))
+      (net 51 "/RX3") (pinfunction "Pin_6") (pintype "passive"))
     (pad "7" thru_hole oval (at 0 7.62 90) (size 1.7 1.7) (drill 1) (layers "*.Cu" "*.Mask")
       (net 49 "/RES0") (pinfunction "Pin_7") (pintype "passive"))
@@
   )
   (footprint "Capacitor_SMD:C_1206_3216Metric" (layer "F.Cu")
+    (at 86.2566 94.361)
+    (descr "Capacitor SMD 1206 (3216 Metric), square (rectangular) end terminal, IPC_7351 nominal, (Body size source: IPC-SM-782 page 76, https://www.pcb-3d.com/wordpress/wp-content/uploads/ipc-sm-782a_amendment_1_and_2.pdf), generated with kicad-footprint-generator")
+    (tags "capacitor")
+    (property "Sheetfile" "RAMROM_Board_v3.kicad_sch")
+    (property "Sheetname" "")
+    (property "ki_description" "Unpolarized capacitor, small symbol")
+    (property "ki_keywords" "capacitor cap")
+    (attr smd)
+    (fp_text reference "C10" (at 0 -1.85) (layer "F.SilkS")
+        (effects (font (size 1 1) (thickness 0.15)))
+    )
+    (fp_text value "100n" (at 0 1.85) (layer "F.Fab")
+        (effects (font (size 1 1) (thickness 0.15)))
+    )
+    (fp_text user "${REFERENCE}" (at 0 0) (layer "F.Fab")
+        (effects (font (size 0.8 0.8) (thickness 0.12)))
+    )
+    (fp_line (start -0.711252 -0.91) (end 0.711252 -0.91)
+      (stroke (width 0.12) (type solid)) (layer "F.SilkS"))
+    (fp_line (start -0.711252 0.91) (end 0.711252 0.91)
+      (stroke (width 0.12) (type solid)) (layer "F.SilkS"))
+    (fp_line (start -2.3 -1.15) (end 2.3 -1.15)
+      (stroke (width 0.05) (type solid)) (layer "F.CrtYd"))
+    (fp_line (start -2.3 1.15) (end -2.3 -1.15)
+      (stroke (width 0.05) (type solid)) (layer "F.CrtYd"))
+    (fp_line (start 2.3 -1.15) (end 2.3 1.15)
+      (stroke (width 0.05) (type solid)) (layer "F.CrtYd"))
+    (fp_line (start 2.3 1.15) (end -2.3 1.15)
+      (stroke (width 0.05) (type solid)) (layer "F.CrtYd"))
+    (fp_line (start -1.6 -0.8) (end 1.6 -0.8)
+      (stroke (width 0.1) (type solid)) (layer "F.Fab"))
+    (fp_line (start -1.6 0.8) (end -1.6 -0.8)
+      (stroke (width 0.1) (type solid)) (layer "F.Fab"))
+    (fp_line (start 1.6 -0.8) (end 1.6 0.8)
+      (stroke (width 0.1) (type solid)) (layer "F.Fab"))
+    (fp_line (start 1.6 0.8) (end -1.6 0.8)
+      (stroke (width 0.1) (type solid)) (layer "F.Fab"))
+    (pad "1" smd roundrect (at -1.475 0) (size 1.15 1.8) (layers "F.Cu" "F.Paste" "F.Mask") (roundrect_rratio 0.217391)
+      (net 31 "+3V3") (pintype "passive"))
+    (pad "2" smd roundrect (at 1.475 0) (size 1.15 1.8) (layers "F.Cu" "F.Paste" "F.Mask") (roundrect_rratio 0.217391)
+      (net 2 "GND") (pintype "passive"))
+    (model "${KICAD6_3DMODEL_DIR}/Capacitor_SMD.3dshapes/C_1206_3216Metric.wrl"
+      (offset (xyz 0 0 0))
+      (scale (xyz 1 1 1))
+      (rotate (xyz 0 0 0))
+    )
+  )
+  (footprint "Capacitor_SMD:C_1206_3216Metric" (layer "F.Cu")
     (at 130.8608 93.853 -90)
     (descr "Capacitor SMD 1206 (3216 Metric), square (rectangular) end terminal, IPC_7351 nominal, (Body size source: IPC-SM-782 page 76, https://www.pcb-3d.com/wordpress/wp-content/uploads/ipc-sm-782a_amendment_1_and_2.pdf), generated with kicad-footprint-generator")
@@
       (net 11 "+5V") (pinfunction "Pin_2") (pintype "passive"))
     (pad "3" thru_hole oval (at 0 2.54 90) (size 1.7 1.7) (drill 1) (layers "*.Cu" "*.Mask")
-      (net 53 "/RX2") (pinfunction "Pin_3") (pintype "passive"))
+      (net 52 "/TX2") (pinfunction "Pin_3") (pintype "passive"))
     (pad "4" thru_hole oval (at -2.54 2.54 90) (size 1.7 1.7) (drill 1) (layers "*.Cu" "*.Mask")
-      (net 52 "/TX2") (pinfunction "Pin_4") (pintype "passive"))
+      (net 53 "/RX2") (pinfunction "Pin_4") (pintype "passive"))
     (pad "5" thru_hole oval (at 0 5.08 90) (size 1.7 1.7) (drill 1) (layers "*.Cu" "*.Mask")
-      (net 51 "/RX3") (pinfunction "Pin_5") (pintype "passive"))
+      (net 50 "/TX3") (pinfunction "Pin_5") (pintype "passive"))
     (pad "6" thru_hole oval (at -2.54 5.08 90) (size 1.7 1.7) (drill 1) (layers "*.Cu" "*.Mask")
-      (net 50 "/TX3") (pinfunction "Pin_6") (pintype "passive"))
+      (net 51 "/RX3") (pinfunction "Pin_6") (pintype "passive"))
     (pad "7" thru_hole oval (at 0 7.62 90) (size 1.7 1.7) (drill 1) (layers "*.Cu" "*.Mask")
       (net 49 "/RES0") (pinfunction "Pin_7") (pintype "passive"))
@@
   (segment (start 146.07 135.099005) (end 147.32 133.849005) (width 0.4) (layer "B.Cu") (net 49))
   (segment (start 147.32 139.7) (end 147.32 138.497919) (width 0.4) (layer "B.Cu") (net 49))
-  (segment (start 144.78 136.017) (end 144.78 137.287) (width 0.4) (layer "B.Cu") (net 50))
-  (segment (start 146.05 138.557) (end 146.05 140.97) (width 0.4) (layer "B.Cu") (net 50))
-  (segment (start 146.05 140.97) (end 144.78 142.24) (width 0.4) (layer "B.Cu") (net 50))
-  (segment (start 144.78 137.287) (end 146.05 138.557) (width 0.4) (layer "B.Cu") (net 50))
-  (segment (start 144.78 134.621238) (end 144.78 133.849005) (width 0.4) (layer "B.Cu") (net 51))
-  (segment (start 143.53 137.18) (end 143.53 135.871238) (width 0.4) (layer "B.Cu") (net 51))
-  (segment (start 143.53 135.871238) (end 144.78 134.621238) (width 0.4) (layer "B.Cu") (net 51))
-  (segment (start 144.78 138.43) (end 143.53 137.18) (width 0.4) (layer "B.Cu") (net 51))
-  (segment (start 144.78 139.623705) (end 144.78 138.43) (width 0.4) (layer "B.Cu") (net 51))
-  (segment (start 143.49 140.99) (end 142.24 142.24) (width 0.4) (layer "B.Cu") (net 52))
-  (segment (start 143.49 138.537) (end 143.49 140.99) (width 0.4) (layer "B.Cu") (net 52))
-  (segment (start 142.24 136.017) (end 142.24 137.287) (width 0.4) (layer "B.Cu") (net 52))
-  (segment (start 142.24 137.287) (end 143.49 138.537) (width 0.4) (layer "B.Cu") (net 52))
-  (segment (start 140.99 138.45) (end 140.99 135.099005) (width 0.4) (layer "B.Cu") (net 53))
-  (segment (start 140.99 135.099005) (end 142.24 133.849005) (width 0.4) (layer "B.Cu") (net 53))
-  (segment (start 142.24 139.7) (end 140.99 138.45) (width 0.4) (layer "B.Cu") (net 53))
+  (segment (start 144.78 134.621238) (end 144.78 133.849005) (width 0.4) (layer "B.Cu") (net 50))
+  (segment (start 143.53 137.18) (end 143.53 135.871238) (width 0.4) (layer "B.Cu") (net 50))
+  (segment (start 143.53 135.871238) (end 144.78 134.621238) (width 0.4) (layer "B.Cu") (net 50))
+  (segment (start 144.78 138.43) (end 143.53 137.18) (width 0.4) (layer "B.Cu") (net 50))
+  (segment (start 144.78 139.623705) (end 144.78 138.43) (width 0.4) (layer "B.Cu") (net 50))
+  (segment (start 144.78 136.017) (end 144.78 137.287) (width 0.4) (layer "B.Cu") (net 51))
+  (segment (start 146.05 138.557) (end 146.05 140.97) (width 0.4) (layer "B.Cu") (net 51))
+  (segment (start 146.05 140.97) (end 144.78 142.24) (width 0.4) (layer "B.Cu") (net 51))
+  (segment (start 144.78 137.287) (end 146.05 138.557) (width 0.4) (layer "B.Cu") (net 51))
+  (segment (start 140.99 138.45) (end 140.99 135.099005) (width 0.4) (layer "B.Cu") (net 52))
+  (segment (start 140.99 135.099005) (end 142.24 133.849005) (width 0.4) (layer "B.Cu") (net 52))
+  (segment (start 142.24 139.7) (end 140.99 138.45) (width 0.4) (layer "B.Cu") (net 52))
+  (segment (start 143.49 140.99) (end 142.24 142.24) (width 0.4) (layer "B.Cu") (net 53))
+  (segment (start 143.49 138.537) (end 143.49 140.99) (width 0.4) (layer "B.Cu") (net 53))
+  (segment (start 142.24 136.017) (end 142.24 137.287) (width 0.4) (layer "B.Cu") (net 53))
+  (segment (start 142.24 137.287) (end 143.49 138.537) (width 0.4) (layer "B.Cu") (net 53))
   (segment (start 177.8 136.779) (end 179.05 138.029) (width 0.4) (layer "B.Cu") (net 54))
   (segment (start 179.05 138.029) (end 179.05 140.99) (width 0.4) (layer "B.Cu") (net 54))
