File: RAMROM_CPLD_board/RAMROM_CPLD_board.kicad_pcb (KiCad board)
At the start: 2 copper layers, 100 x 100 mm, 46 parts, among them J1 BUS, J10 CS_Breakout, J106 Conn_01x32, J107 Conn_01x32, J108 Conn_01x38_Male, J109 Conn_01x38_Male, J11 BO2, J110 Conn_01x38_Male, J18 Conn_01x38_Male, J2 Conn_01x07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

Commit message: Readme update
Connections:
- J1 pad 3: /TX2 -> /RX2
- J1 pad 4: /RX2 -> /TX2
- J1 pad 5: /TX3 -> /RX3
- J1 pad 6: /RX3 -> /TX3
- J11 pad 1: /RX2 -> /TX2
- J11 pad 2: /TX2 -> /RX2
- J11 pad 3: /RX3 -> /TX3
- J11 pad 4: /TX3 -> /RX3
Routing:
- net /RX2: track 36.3 -> 32.9 mm
