File: RAMROM_CPLD_board/RAMROM_CPLD_board.kicad_sch (KiCad schematic)
At the start: 27 parts, among them J1 BUS, J10 CS_Breakout, J11 BO2, J2 Conn_01x07, J26 STM32F411, J3 BUS, J4 Conn_02x07_Counter_Clockwise, J5 Conn_01x07, J7 Conn_01x13, J8 Conn_01x03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

Commit message: Readme update
Connections:
- net RX2: now also J1.3 (Pin_3), J11.2 (Pin_2); no longer J1.4 (Pin_4), J11.1 (Pin_1)
- net RX3: now also J1.5 (Pin_5), J11.4 (Pin_4); no longer J1.6 (Pin_6), J11.3 (Pin_3)
- net TX2: now also J1.4 (Pin_4), J11.1 (Pin_1); no longer J1.3 (Pin_3), J11.2 (Pin_2)
- net TX3: now also J1.6 (Pin_6), J11.3 (Pin_3); no longer J1.5 (Pin_5), J11.4 (Pin_4)
