File: empty_CPU_board_w_CPLD/bus.kicad_sch (KiCad schematic)
At the start: 6 parts

Commit message: Readme update
Connections:
- net RX2: now also J?.3 (Pin_3), J?.3 (Pin_3); no longer J?.4 (Pin_4), J?.4 (Pin_4)
- net RX3: now also J?.5 (Pin_5), J?.5 (Pin_5); no longer J?.6 (Pin_6), J?.6 (Pin_6)
- net TX2: now also J?.4 (Pin_4), J?.4 (Pin_4); no longer J?.3 (Pin_3), J?.3 (Pin_3)
- net TX3: now also J?.6 (Pin_6), J?.6 (Pin_6); no longer J?.5 (Pin_5), J?.5 (Pin_5)
Changed lines of the file:
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@@
     (effects (font (size 1.27 1.27)) (justify left bottom))
   )
-  (label "RX3" (at 99.695 96.52 180) (fields_autoplaced)
-    (effects (font (size 1.27 1.27)) (justify right bottom))
+  (label "RX3" (at 61.595 96.52 0) (fields_autoplaced)
+    (effects (font (size 1.27 1.27)) (justify left bottom))
   )
   (label "A8" (at 128.27 59.69 0) (fields_autoplaced)
@@
     (effects (font (size 1.27 1.27)) (justify left bottom))
   )
-  (label "RX2" (at 99.695 93.98 180) (fields_autoplaced)
-    (effects (font (size 1.27 1.27)) (justify right bottom))
+  (label "RX2" (at 61.595 93.98 0) (fields_autoplaced)
+    (effects (font (size 1.27 1.27)) (justify left bottom))
   )
   (label "A14" (at 128.27 67.31 0) (fields_autoplaced)
@@
     (effects (font (size 1.27 1.27)) (justify right bottom))
   )
-  (label "TX3" (at 61.595 96.52 0) (fields_autoplaced)
-    (effects (font (size 1.27 1.27)) (justify left bottom))
+  (label "TX3" (at 99.695 96.52 180) (fields_autoplaced)
+    (effects (font (size 1.27 1.27)) (justify right bottom))
   )
   (label "A2" (at 128.27 52.07 0) (fields_autoplaced)
@@
     (effects (font (size 1.27 1.27)) (justify left bottom))
   )
-  (label "TX2" (at 61.595 93.98 0) (fields_autoplaced)
-    (effects (font (size 1.27 1.27)) (justify left bottom))
+  (label "TX2" (at 99.695 93.98 180) (fields_autoplaced)
+    (effects (font (size 1.27 1.27)) (justify right bottom))
   )
   (label "A19" (at 39.37 74.295 180) (fields_autoplaced)
@@
     (effects (font (size 1.27 1.27)) (justify right))
   )
-  (hierarchical_label "TX2" (shape output) (at 121.285 93.98 180) (fields_autoplaced)
-    (effects (font (size 1.27 1.27)) (justify right))
+  (hierarchical_label "TX2" (shape output) (at 160.655 93.98 0) (fields_autoplaced)
+    (effects (font (size 1.27 1.27)) (justify left))
   )
   (hierarchical_label "SCK" (shape output) (at 125.73 129.54 180) (fields_autoplaced)
@@
     (effects (font (size 1.27 1.27)) (justify left))
   )
-  (hierarchical_label "RX2" (shape input) (at 160.655 93.98 0) (fields_autoplaced)
-    (effects (font (size 1.27 1.27)) (justify left))
+  (hierarchical_label "RX2" (shape input) (at 121.285 93.98 180) (fields_autoplaced)
+    (effects (font (size 1.27 1.27)) (justify right))
   )
   (hierarchical_label "~{RST}" (shape bidirectional) (at 156.21 46.99 0) (fields_autoplaced)
@@
     (effects (font (size 1.27 1.27)) (justify right))
   )
-  (hierarchical_label "RX3" (shape input) (at 160.655 96.52 0) (fields_autoplaced)
-    (effects (font (size 1.27 1.27)) (justify left))
+  (hierarchical_label "RX3" (shape input) (at 121.285 96.52 180) (fields_autoplaced)
+    (effects (font (size 1.27 1.27)) (justify right))
   )
   (hierarchical_label "R{slash}~{W}_e" (shape output) (at 151.13 31.75 0) (fields_autoplaced)
@@
     (effects (font (size 1.27 1.27)) (justify left))
   )
-  (hierarchical_label "TX3" (shape input) (at 121.285 96.52 180) (fields_autoplaced)
-    (effects (font (size 1.27 1.27)) (justify right))
+  (hierarchical_label "TX3" (shape output) (at 160.655 96.52 0) (fields_autoplaced)
+    (effects (font (size 1.27 1.27)) (justify left))
   )
   (hierarchical_label "CLKF" (shape output) (at 160.655 106.68 0) (fields_autoplaced)
