File: empty_board_w_mapping_ram2/bus.kicad_sch (KiCad schematic)
At the start: 4 parts

Commit message: Readme update
Connections:
- net RX2: now also J?.3 (Pin_3), J?.3 (Pin_3); no longer J?.4 (Pin_4), J?.4 (Pin_4)
- net RX3: now also J?.5 (Pin_5), J?.5 (Pin_5); no longer J?.6 (Pin_6), J?.6 (Pin_6)
- net TX2: now also J?.4 (Pin_4), J?.4 (Pin_4); no longer J?.3 (Pin_3), J?.3 (Pin_3)
- net TX3: now also J?.6 (Pin_6), J?.6 (Pin_6); no longer J?.5 (Pin_5), J?.5 (Pin_5)
Changed lines of the file:
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@@
     (effects (font (size 1.27 1.27)) (justify left bottom))
   )
-  (label "TX3" (at 62.865 95.25 0) (fields_autoplaced)
-    (effects (font (size 1.27 1.27)) (justify left bottom))
+  (label "TX3" (at 100.965 95.25 180) (fields_autoplaced)
+    (effects (font (size 1.27 1.27)) (justify right bottom))
   )
   (label "PH0" (at 62.865 102.87 0) (fields_autoplaced)
@@
     (effects (font (size 1.27 1.27)) (justify left bottom))
   )
-  (label "TX2" (at 62.865 92.71 0) (fields_autoplaced)
-    (effects (font (size 1.27 1.27)) (justify left bottom))
+  (label "TX2" (at 100.965 92.71 180) (fields_autoplaced)
+    (effects (font (size 1.27 1.27)) (justify right bottom))
   )
   (label "~{RAMWE9}" (at 182.88 116.84 0) (fields_autoplaced)
@@
     (effects (font (size 1.27 1.27)) (justify left bottom))
   )
-  (label "RX3" (at 100.965 95.25 180) (fields_autoplaced)
-    (effects (font (size 1.27 1.27)) (justify right bottom))
+  (label "RX3" (at 62.865 95.25 0) (fields_autoplaced)
+    (effects (font (size 1.27 1.27)) (justify left bottom))
   )
   (label "~{MWR}" (at 104.14 34.29 180) (fields_autoplaced)
@@
     (effects (font (size 1.27 1.27)) (justify left bottom))
   )
-  (label "RX2" (at 100.965 92.71 180) (fields_autoplaced)
-    (effects (font (size 1.27 1.27)) (justify right bottom))
+  (label "RX2" (at 62.865 92.71 0) (fields_autoplaced)
+    (effects (font (size 1.27 1.27)) (justify left bottom))
   )
   (label "A18" (at 39.37 71.755 180) (fields_autoplaced)
@@
     (effects (font (size 1.27 1.27)) (justify left))
   )
-  (hierarchical_label "RX2" (shape input) (at 161.925 92.71 0) (fields_autoplaced)
-    (effects (font (size 1.27 1.27)) (justify left))
+  (hierarchical_label "RX2" (shape input) (at 122.555 92.71 180) (fields_autoplaced)
+    (effects (font (size 1.27 1.27)) (justify right))
   )
   (hierarchical_label "MOSI" (shape output) (at 161.925 125.73 0) (fields_autoplaced)
@@
     (effects (font (size 1.27 1.27)) (justify left))
   )
-  (hierarchical_label "TX3" (shape input) (at 122.555 95.25 180) (fields_autoplaced)
-    (effects (font (size 1.27 1.27)) (justify right))
+  (hierarchical_label "TX3" (shape output) (at 161.925 95.25 0) (fields_autoplaced)
+    (effects (font (size 1.27 1.27)) (justify left))
   )
   (hierarchical_label "TMS" (shape output) (at 127 130.81 180) (fields_autoplaced)
@@
     (effects (font (size 1.27 1.27)) (justify left))
   )
-  (hierarchical_label "RX3" (shape input) (at 161.925 95.25 0) (fields_autoplaced)
-    (effects (font (size 1.27 1.27)) (justify left))
+  (hierarchical_label "RX3" (shape input) (at 122.555 95.25 180) (fields_autoplaced)
+    (effects (font (size 1.27 1.27)) (justify right))
   )
   (hierarchical_label "TDO" (shape output) (at 156.845 130.81 0) (fields_autoplaced)
@@
     (effects (font (size 1.27 1.27)) (justify right))
   )
-  (hierarchical_label "TX2" (shape output) (at 122.555 92.71 180) (fields_autoplaced)
-    (effects (font (size 1.27 1.27)) (justify right))
+  (hierarchical_label "TX2" (shape output) (at 161.925 92.71 0) (fields_autoplaced)
+    (effects (font (size 1.27 1.27)) (justify left))
   )
   (hierarchical_label "R{slash}~{W}_e" (shape output) (at 151.13 31.75 0) (fields_autoplaced)
