File: empty_board_w_mapping_ram2/empty_board_w_mapping_ram2.kicad_sch (KiCad schematic)
At the start: 21 parts, among them J10 ., J11 ., J8 ., U1 SN74LVC245ANSR, U2 74HC14, U5 IS63WV1288DBLL-10xLI, U6 74LVC253, U7 74LVC595, U8 74AHC1G14

Commit message: Readme update
Changed lines of the file:
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@@
     (effects (font (size 1.27 1.27)) (justify left bottom))
   )
-  (label "TX2" (at 14.605 46.355 0) (fields_autoplaced)
+  (label "TX2" (at 14.605 43.815 0) (fields_autoplaced)
     (effects (font (size 1.27 1.27)) (justify left bottom))
   )
@@
     (effects (font (size 1.27 1.27)) (justify left bottom))
   )
-  (label "TX3" (at 14.605 51.435 0) (fields_autoplaced)
+  (label "TX3" (at 14.605 48.895 0) (fields_autoplaced)
     (effects (font (size 1.27 1.27)) (justify left bottom))
   )
@@
     (effects (font (size 1.27 1.27)) (justify left bottom))
   )
-  (label "RX3" (at 14.605 48.895 0) (fields_autoplaced)
+  (label "RX3" (at 14.605 51.435 0) (fields_autoplaced)
     (effects (font (size 1.27 1.27)) (justify left bottom))
   )
@@
     (effects (font (size 1.27 1.27)) (justify left bottom))
   )
-  (label "RX2" (at 14.605 43.815 0) (fields_autoplaced)
+  (label "RX2" (at 14.605 46.355 0) (fields_autoplaced)
     (effects (font (size 1.27 1.27)) (justify left bottom))
   )
