File: MultiSerial v2/schematic/MOS MultiSerial_ram/MOS MultiSerial_ram.kicad_pcb (KiCad board)
At the start: 2 copper layers, 100 x 100 mm, 48 parts, among them J1 BUS, J12 Conn_01x01, J13 Conn_01x04, J14 Conn_01x02, J15 Conn_02x36_Counter_Clockwise, J16 Conn_02x36_Counter_Clockwise, J17 Conn_02x36_Counter_Clockwise, J18 Conn_02x36_Counter_Clockwise, J19 Conn_02x36_Counter_Clockwise, J2 BUS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

Commit message: Readme update
Connections:
- J2 pad 3: /RX2 -> /TX2
- J2 pad 4: /TX2 -> /RX2
- J2 pad 5: /RX3 -> /TX3
- J2 pad 6: /TX3 -> /RX3
- J4 pad 3: /RX2 -> /TX2
- J4 pad 4: /TX2 -> /RX2
- J4 pad 5: /RX3 -> /TX3
- J4 pad 6: /TX3 -> /RX3
Changed lines of the file:
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@@
       (net 11 "+5V") (pinfunction "Pin_2") (pintype "passive"))
     (pad "3" thru_hole oval (at 0 2.54 90) (size 1.7 1.7) (drill 1) (layers "*.Cu" "*.Mask")
-      (net 53 "/RX2") (pinfunction "Pin_3") (pintype "passive"))
+      (net 52 "/TX2") (pinfunction "Pin_3") (pintype "passive"))
     (pad "4" thru_hole oval (at -2.54 2.54 90) (size 1.7 1.7) (drill 1) (layers "*.Cu" "*.Mask")
-      (net 52 "/TX2") (pinfunction "Pin_4") (pintype "passive"))
+      (net 53 "/RX2") (pinfunction "Pin_4") (pintype "passive"))
     (pad "5" thru_hole oval (at 0 5.08 90) (size 1.7 1.7) (drill 1) (layers "*.Cu" "*.Mask")
-      (net 51 "/RX3") (pinfunction "Pin_5") (pintype "passive"))
+      (net 50 "/TX3") (pinfunction "Pin_5") (pintype "passive"))
     (pad "6" thru_hole oval (at -2.54 5.08 90) (size 1.7 1.7) (drill 1) (layers "*.Cu" "*.Mask")
-      (net 50 "/TX3") (pinfunction "Pin_6") (pintype "passive"))
+      (net 51 "/RX3") (pinfunction "Pin_6") (pintype "passive"))
     (pad "7" thru_hole oval (at 0 7.62 90) (size 1.7 1.7) (drill 1) (layers "*.Cu" "*.Mask")
       (net 49 "/RES0") (pinfunction "Pin_7") (pintype "passive"))
@@
       (net 11 "+5V") (pinfunction "Pin_2") (pintype "passive"))
     (pad "3" thru_hole oval (at 0 2.54 90) (size 1.7 1.7) (drill 1) (layers "*.Cu" "*.Mask")
-      (net 53 "/RX2") (pinfunction "Pin_3") (pintype "passive"))
+      (net 52 "/TX2") (pinfunction "Pin_3") (pintype "passive"))
     (pad "4" thru_hole oval (at -2.54 2.54 90) (size 1.7 1.7) (drill 1) (layers "*.Cu" "*.Mask")
-      (net 52 "/TX2") (pinfunction "Pin_4") (pintype "passive"))
+      (net 53 "/RX2") (pinfunction "Pin_4") (pintype "passive"))
     (pad "5" thru_hole oval (at 0 5.08 90) (size 1.7 1.7) (drill 1) (layers "*.Cu" "*.Mask")
-      (net 51 "/RX3") (pinfunction "Pin_5") (pintype "passive"))
+      (net 50 "/TX3") (pinfunction "Pin_5") (pintype "passive"))
     (pad "6" thru_hole oval (at -2.54 5.08 90) (size 1.7 1.7) (drill 1) (layers "*.Cu" "*.Mask")
-      (net 50 "/TX3") (pinfunction "Pin_6") (pintype "passive"))
+      (net 51 "/RX3") (pinfunction "Pin_6") (pintype "passive"))
     (pad "7" thru_hole oval (at 0 7.62 90) (size 1.7 1.7) (drill 1) (layers "*.Cu" "*.Mask")
       (net 49 "/RES0") (pinfunction "Pin_7") (pintype "passive"))
@@
   (segment (start 146.07 135.099005) (end 147.32 133.849005) (width 0.4) (layer "B.Cu") (net 49))
   (segment (start 147.32 139.7) (end 147.32 138.497919) (width 0.4) (layer "B.Cu") (net 49))
-  (segment (start 144.78 136.017) (end 144.78 137.287) (width 0.4) (layer "B.Cu") (net 50))
-  (segment (start 146.05 138.557) (end 146.05 140.97) (width 0.4) (layer "B.Cu") (net 50))
-  (segment (start 146.05 140.97) (end 144.78 142.24) (width 0.4) (layer "B.Cu") (net 50))
-  (segment (start 144.78 137.287) (end 146.05 138.557) (width 0.4) (layer "B.Cu") (net 50))
-  (segment (start 144.78 134.621238) (end 144.78 133.849005) (width 0.4) (layer "B.Cu") (net 51))
-  (segment (start 143.53 137.18) (end 143.53 135.871238) (width 0.4) (layer "B.Cu") (net 51))
-  (segment (start 143.53 135.871238) (end 144.78 134.621238) (width 0.4) (layer "B.Cu") (net 51))
-  (segment (start 144.78 138.43) (end 143.53 137.18) (width 0.4) (layer "B.Cu") (net 51))
-  (segment (start 144.78 139.623705) (end 144.78 138.43) (width 0.4) (layer "B.Cu") (net 51))
-  (segment (start 143.49 140.99) (end 142.24 142.24) (width 0.4) (layer "B.Cu") (net 52))
-  (segment (start 143.49 138.537) (end 143.49 140.99) (width 0.4) (layer "B.Cu") (net 52))
-  (segment (start 142.24 136.017) (end 142.24 137.287) (width 0.4) (layer "B.Cu") (net 52))
-  (segment (start 142.24 137.287) (end 143.49 138.537) (width 0.4) (layer "B.Cu") (net 52))
-  (segment (start 140.99 138.45) (end 140.99 135.099005) (width 0.4) (layer "B.Cu") (net 53))
-  (segment (start 140.99 135.099005) (end 142.24 133.849005) (width 0.4) (layer "B.Cu") (net 53))
-  (segment (start 142.24 139.7) (end 140.99 138.45) (width 0.4) (layer "B.Cu") (net 53))
+  (segment (start 144.78 134.621238) (end 144.78 133.849005) (width 0.4) (layer "B.Cu") (net 50))
+  (segment (start 143.53 137.18) (end 143.53 135.871238) (width 0.4) (layer "B.Cu") (net 50))
+  (segment (start 143.53 135.871238) (end 144.78 134.621238) (width 0.4) (layer "B.Cu") (net 50))
+  (segment (start 144.78 138.43) (end 143.53 137.18) (width 0.4) (layer "B.Cu") (net 50))
+  (segment (start 144.78 139.623705) (end 144.78 138.43) (width 0.4) (layer "B.Cu") (net 50))
+  (segment (start 144.78 136.017) (end 144.78 137.287) (width 0.4) (layer "B.Cu") (net 51))
+  (segment (start 146.05 138.557) (end 146.05 140.97) (width 0.4) (layer "B.Cu") (net 51))
+  (segment (start 146.05 140.97) (end 144.78 142.24) (width 0.4) (layer "B.Cu") (net 51))
+  (segment (start 144.78 137.287) (end 146.05 138.557) (width 0.4) (layer "B.Cu") (net 51))
+  (segment (start 140.99 138.45) (end 140.99 135.099005) (width 0.4) (layer "B.Cu") (net 52))
+  (segment (start 140.99 135.099005) (end 142.24 133.849005) (width 0.4) (layer "B.Cu") (net 52))
+  (segment (start 142.24 139.7) (end 140.99 138.45) (width 0.4) (layer "B.Cu") (net 52))
+  (segment (start 143.49 140.99) (end 142.24 142.24) (width 0.4) (layer "B.Cu") (net 53))
+  (segment (start 143.49 138.537) (end 143.49 140.99) (width 0.4) (layer "B.Cu") (net 53))
+  (segment (start 142.24 136.017) (end 142.24 137.287) (width 0.4) (layer "B.Cu") (net 53))
+  (segment (start 142.24 137.287) (end 143.49 138.537) (width 0.4) (layer "B.Cu") (net 53))
   (segment (start 177.8 136.779) (end 179.05 138.029) (width 0.4) (layer "B.Cu") (net 54))
   (segment (start 179.05 138.029) (end 179.05 140.99) (width 0.4) (layer "B.Cu") (net 54))

Commit message: python work
Parts:
- added J24: Conn_01x01, Connector_PinHeader_2.00mm:PinHeader_1x01_P2.00mm_Vertical, F.Cu at (167.8, 62.0)
- added U10: 74AHC1G08, Package_TO_SOT_SMD:SOT-23-5_HandSoldering, F.Cu at (161.7, 64.1)
Connections:
- J2 pad 3: /TX2 -> /RX2
- J2 pad 4: /RX2 -> /TX2
- J2 pad 5: /TX3 -> /RX3
- J2 pad 6: /RX3 -> /TX3
- J22 pad 1: /PHI2_e -> /Bus/~{DOE}
- J4 pad 3: /TX2 -> /RX2
- J4 pad 4: /RX2 -> /TX2
- J4 pad 5: /TX3 -> /RX3
- J4 pad 6: /RX3 -> /TX3
- U9 pad 22: /PHI2_e -> /Bus/~{DOE}
Routing:
- net GND: track 568.2 -> 610.0 mm, vias 10 -> 12
- net /PHI2_e: track 36.0 -> 13.2 mm
- net /Bus/~{DOE}: track 0.00 -> 18.6 mm, vias 0 -> 1
- net +3V3: track 320.6 -> 326.0 mm, vias 3 -> 4
- net /~{CS_ACIA2}: track 38.5 -> 43.1 mm, vias 1 -> 0
- net /~{CS_ACIA}: track 95.0 -> 98.6 mm
- net +5V: track 230.7 -> 227.5 mm
- net /~{RST}: track 105.7 -> 107.7 mm
