File: MultiSerial v2/schematic/MOS MultiSerial_ram/bus.kicad_sch (KiCad schematic)
At the start: 8 parts, among them J12 Conn_01x01, U1 SN74LVCC4245ANSR

Commit message: Readme update
Connections:
- net RX2: now also J?.3 (Pin_3), J?.3 (Pin_3); no longer J?.4 (Pin_4), J?.4 (Pin_4)
- net RX3: now also J?.5 (Pin_5), J?.5 (Pin_5); no longer J?.6 (Pin_6), J?.6 (Pin_6)
- net TX2: now also J?.4 (Pin_4), J?.4 (Pin_4); no longer J?.3 (Pin_3), J?.3 (Pin_3)
- net TX3: now also J?.6 (Pin_6), J?.6 (Pin_6); no longer J?.5 (Pin_5), J?.5 (Pin_5)
Changed lines of the file:
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@@
     (effects (font (size 1.27 1.27)) (justify left bottom))
   )
-  (label "RX3" (at 100.33 97.79 180) (fields_autoplaced)
-    (effects (font (size 1.27 1.27)) (justify right bottom))
+  (label "RX3" (at 62.23 97.79 0) (fields_autoplaced)
+    (effects (font (size 1.27 1.27)) (justify left bottom))
   )
   (label "DB5" (at 239.395 47.625 180) (fields_autoplaced)
@@
     (effects (font (size 1.27 1.27)) (justify right bottom))
   )
-  (label "TX2" (at 62.23 95.25 0) (fields_autoplaced)
-    (effects (font (size 1.27 1.27)) (justify left bottom))
+  (label "TX2" (at 100.33 95.25 180) (fields_autoplaced)
+    (effects (font (size 1.27 1.27)) (justify right bottom))
   )
   (label "RES1" (at 62.23 102.87 0) (fields_autoplaced)
@@
     (effects (font (size 1.27 1.27)) (justify left bottom))
   )
-  (label "RX2" (at 100.33 95.25 180) (fields_autoplaced)
-    (effects (font (size 1.27 1.27)) (justify right bottom))
+  (label "RX2" (at 62.23 95.25 0) (fields_autoplaced)
+    (effects (font (size 1.27 1.27)) (justify left bottom))
   )
   (label "~{RAMWE5}" (at 182.245 109.22 0) (fields_autoplaced)
     (effects (font (size 1.27 1.27)) (justify left bottom))
   )
-  (label "TX3" (at 62.23 97.79 0) (fields_autoplaced)
-    (effects (font (size 1.27 1.27)) (justify left bottom))
+  (label "TX3" (at 100.33 97.79 180) (fields_autoplaced)
+    (effects (font (size 1.27 1.27)) (justify right bottom))
   )
   (label "SCK" (at 62.23 130.81 0) (fields_autoplaced)
@@
     (effects (font (size 1.27 1.27)) (justify right))
   )
-  (hierarchical_label "RX3" (shape input) (at 161.29 97.79 0) (fields_autoplaced)
-    (effects (font (size 1.27 1.27)) (justify left))
+  (hierarchical_label "RX3" (shape input) (at 121.92 97.79 180) (fields_autoplaced)
+    (effects (font (size 1.27 1.27)) (justify right))
   )
   (hierarchical_label "CLKS" (shape output) (at 121.92 107.95 180) (fields_autoplaced)
@@
     (effects (font (size 1.27 1.27)) (justify left))
   )
-  (hierarchical_label "TX3" (shape input) (at 121.92 97.79 180) (fields_autoplaced)
-    (effects (font (size 1.27 1.27)) (justify right))
+  (hierarchical_label "TX3" (shape output) (at 161.29 97.79 0) (fields_autoplaced)
+    (effects (font (size 1.27 1.27)) (justify left))
   )
   (hierarchical_label "CLKF" (shape output) (at 161.29 107.95 0) (fields_autoplaced)
@@
     (effects (font (size 1.27 1.27)) (justify right))
   )
-  (hierarchical_label "TX2" (shape output) (at 121.92 95.25 180) (fields_autoplaced)
-    (effects (font (size 1.27 1.27)) (justify right))
+  (hierarchical_label "TX2" (shape output) (at 161.29 95.25 0) (fields_autoplaced)
+    (effects (font (size 1.27 1.27)) (justify left))
   )
   (hierarchical_label "~{RAMWE[0..13]}" (shape output) (at 201.295 92.71 0) (fields_autoplaced)
     (effects (font (size 1.27 1.27)) (justify left))
   )
-  (hierarchical_label "RX2" (shape input) (at 161.29 95.25 0) (fields_autoplaced)
-    (effects (font (size 1.27 1.27)) (justify left))
+  (hierarchical_label "RX2" (shape input) (at 121.92 95.25 180) (fields_autoplaced)
+    (effects (font (size 1.27 1.27)) (justify right))
   )
   (symbol (lib_id "power:+5V") (at 128.905 90.805 0) (unit 1)

Commit message: python work
Other:
- moved on the sheet: J12, U1
