File: MultiParallel v2/schematic/MOS_MultiParallel_2/MOS_MultiParallel_2-backups/MOS_MultiParallel_2-2023-07-27_120041/MOS_MultiParallel_2.kicad_pcb (KiCad board)
At the start: 2 copper layers, 100 x 100 mm, 65 parts, among them J1 BUS, J10 ., J11 ., J12 Conn_01x01, J13 ., J14 ., J15 ., J16 ., J17 Conn_01x01, J18 Conn_01x01, J2 BUS, J20 Conn_01x12, J21 Conn_01x12, J25 ., J26 .Conn_01x01, J27 ., J28 ., J29 ., J3 BUS, J30 ., J31 Conn_02x22_Odd_Even, J4 BUS, J5 ., J6 ., J7 ., J8 ., J9 Conn_01x01, U1 SN74LVCC4245ANSR, U11 W65C22NxP, U2 74HC14, U3 6532, U4 W65C22NxP, U5 IS63WV1288DBLL-10xLI, U6 74LVC253, U7 74LVC595, U8 74AHC1G14, U9 74AHC1G08

Commit message: apple I test
Parts:
- removed U9: 74AHC1G08, Package_TO_SOT_SMD:SOT-23-5_HandSoldering
Connections:
- J18 pad 1: /Bus/~{DOE} -> /PHI2_e
- J2 pad 3: /RX2 -> /TX2
- J2 pad 4: /TX2 -> /RX2
- J2 pad 5: /RX3 -> /TX3
- J2 pad 6: /TX3 -> /RX3
- J4 pad 3: /RX2 -> /TX2
- J4 pad 4: /TX2 -> /RX2
- J4 pad 5: /RX3 -> /TX3
- J4 pad 6: /TX3 -> /RX3
- U1 pad 22: /Bus/~{DOE} -> /PHI2_e
Routing:
- net /PHI2_e: track 12.8 -> 48.1 mm, vias 0 -> 1
- net /Bus/~{DOE}: track 33.0 -> 0.00 mm, vias 1 -> 0
- net GND: track 535.0 -> 524.1 mm, vias 7 -> 5
- net +3V3: track 372.3 -> 364.9 mm, vias 4 -> 3
- net /~{CSPIA}: track 123.7 -> 120.3 mm
- net /~{CSPIA2}: track 120.9 -> 122.6 mm
- net Net-(U5-I/O4): track 24.3 -> 23.2 mm
- net Net-(U5-I/O5): track 27.0 -> 26.3 mm
Other:
- board text added: "*Unicomp v2* MOS Multi Parallel Board v1"
- board text removed: "*Unicomp v2* MOS Multi Parallel Board v1.1"
