File: MultiParallel v2/schematic/MOS_MultiParallel_2/MOS_MultiParallel_2-backups/MOS_MultiParallel_2-2023-07-27_120041/MOS_MultiParallel_2.kicad_sch (KiCad schematic)
At the start: 56 parts, among them J10 ., J11 ., J12 Conn_01x01, J13 ., J14 ., J15 ., J16 ., J25 ., J26 .Conn_01x01, J27 .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

Commit message: apple I test
Parts:
- removed U9: 74AHC1G08, Package_TO_SOT_SMD:SOT-23-5_HandSoldering, symbol 74xGxx:74AHC1G08
Other:
- moved on the sheet: A1, C4, J10, J11, J26, J27, J28, J29, J30, J5, J6, J7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
