File: RAMROM_512k_board/RAMROM_512k_board.kicad_sch (KiCad schematic)
At the start: 42 parts, among them J6 STM32F411, J7 ., J8 ., J9 ., Q1 PMV450ENEAR, U1 SN74LVC245ANSR, U10 74LVC595, U12 74AHC1G14, U16 74LVC138, U17 74LVC138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

Commit message: Readme update
Connections:
- net uA9: no longer J6.6 (Pin_6)
- net ~{uMWR}: now also J6.6 (Pin_6); no longer J6.9 (Pin_9)
- new net uA12: J6.9 (Pin_9)
Other:
- note added: "USB"
Changed lines of the file:
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@@
     (title "Unicomp v2 - RAMROM Board")
     (date "2023-07-06")
-    (rev "v1")
+    (rev "v1.1")
     (company "100% Offner")
     (comment 1 "v1: Initial")
+    (comment 2 "v1.1: ~{uMWR} from A12 to A9 of STM32 bec. USB")
   )
   (junction (at 78.105 154.94) (diameter 0) (color 0 0 0 0)
@@
     (stroke (width 0) (type default))
   )
+  (text "USB" (at 19.05 210.185 0)
+    (effects (font (size 1.27 1.27)) (justify left bottom))
+  )
   (text "B1\nB0" (at 60.325 204.47 0)
     (effects (font (size 1.27 1.27)) (justify left bottom))
@@
     (effects (font (size 1.55 1.55)) (justify left bottom))
   )
+  (text "USB" (at 19.05 207.645 0)
+    (effects (font (size 1.27 1.27)) (justify left bottom))
+  )
   (text "B12\nB13\nB14\nB15" (at 25.146 197.866 0)
     (effects (font (size 1.55 1.55)) (justify left bottom))
@@
     (effects (font (size 1.27 1.27)) (justify right bottom))
   )
+  (label "uA12" (at 31.115 210.185 0) (fields_autoplaced)
+    (effects (font (size 1.27 1.27)) (justify left bottom))
+  )
   (label "B2" (at 59.055 200.025 180) (fields_autoplaced)
     (effects (font (size 1.27 1.27)) (justify right bottom))
@@
     (effects (font (size 1.27 1.27)) (justify left bottom))
   )
-  (label "TX2" (at 14.605 46.355 0) (fields_autoplaced)
+  (label "TX2" (at 14.605 43.815 0) (fields_autoplaced)
     (effects (font (size 1.27 1.27)) (justify left bottom))
   )
@@
     (effects (font (size 1.27 1.27)) (justify left bottom))
   )
-  (label "TX3" (at 14.605 51.435 0) (fields_autoplaced)
-    (effects (font (size 1.27 1.27)) (justify left bottom))
-  )
-  (label "uA9" (at 31.115 202.565 0) (fields_autoplaced)
+  (label "TX3" (at 14.605 48.895 0) (fields_autoplaced)
     (effects (font (size 1.27 1.27)) (justify left bottom))
   )
@@
     (effects (font (size 1.27 1.27)) (justify left bottom))
   )
-  (label "RX3" (at 14.605 48.895 0) (fields_autoplaced)
+  (label "RX3" (at 14.605 51.435 0) (fields_autoplaced)
     (effects (font (size 1.27 1.27)) (justify left bottom))
   )
@@
     (effects (font (size 1.27 1.27)) (justify left bottom))
   )
-  (label "RX2" (at 14.605 43.815 0) (fields_autoplaced)
+  (label "RX2" (at 14.605 46.355 0) (fields_autoplaced)
     (effects (font (size 1.27 1.27)) (justify left bottom))
   )
@@
     (effects (font (size 1.27 1.27)) (justify right bottom))
   )
-  (label "~{uMWR}" (at 31.115 210.185 0) (fields_autoplaced)
-    (effects (font (size 1.27 1.27)) (justify left bottom))
-  )
+  (label "~{uMWR}" (at 31.115 202.565 0) (fields_autoplaced)
+    (effects (font (size 1.27 1.27)) (justify left bottom))
+  )

Commit message: Readme update
Parts:
- added U3: 74LVC1G32, Package_TO_SOT_SMD:SOT-23-5_HandSoldering, symbol 74xGxx:74LVC1G32
Connections:
- net +3V3: now also U3.5 (VCC)
- net GND: now also U3.3 (GND)
- net ~{MWR}: now also U3.1
- net at U21.1: now also U3.4; no longer U21.11
- net B10 renamed TRST
- net ~{WP} renamed WP
- net WP: now also U3.2
- no-connect marks 14 -> 15
Other:
- note added: "B10 (B11 on F103) B2 (TRST on F103)"
- note added: "Chip Select Numbers: ~{RAMWE0} - ~{RAMWE13} external Use for Peripherals ~{RAMWE14} - RAMROM Card Enable ~{RAMWE15} - RAMROM Card RAMA Fill"
- note added: "U21D is wrong, it should be a OR Gate."
- note added: "WP is LOW for RAM and High for ROM."
- note removed: "B10 (B11 on F103) B2 (B10 on F103)"
- note removed: "Chip Select Numbers: ~{RAMWE0} - ~{RAMWE14} external Use for Peripherals ~{RAMWE15} - RAMROM Card"
- note removed: "~{WP} is LOW for RAM and High for ROM."
Changed lines of the file:
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@@
     (title "Unicomp v2 - RAMROM Board")
     (date "2023-07-06")
-    (rev "v1.1")
+    (rev "v1.2")
     (company "100% Offner")
     (comment 1 "v1: Initial")
     (comment 2 "v1.1: ~{uMWR} from A12 to A9 of STM32 bec. USB")
+    (comment 3 "v1.2: WP doesnt work, changed to OR-Gate U3.")
   )
   (junction (at 78.105 154.94) (diameter 0) (color 0 0 0 0)
@@
   (no_connect (at 259.08 250.19))
   (no_connect (at 50.8 189.865))
+  (no_connect (at 91.44 111.76))
   (no_connect (at 38.1 238.125))
   (no_connect (at 232.41 45.72))
@@
     (stroke (width 0) (type default))
   )
+  (wire (pts (xy 69.215 138.43) (xy 78.74 138.43))
+    (stroke (width 0) (type default))
+  )
   (wire (pts (xy 149.86 18.415) (xy 149.86 21.59))
     (stroke (width 0) (type default))
@@
     (stroke (width 0) (type default))
   )
-  (wire (pts (xy 93.345 128.905) (xy 91.44 128.905))
+  (wire (pts (xy 78.74 128.905) (xy 93.345 128.905))
     (stroke (width 0) (type default))
   )
@@
     (stroke (width 0) (type default))
   )
-  (wire (pts (xy 91.44 128.905) (xy 91.44 111.76))
-    (stroke (width 0) (type default))
-  )
   (wire (pts (xy 31.115 207.645) (xy 38.1 207.645))
     (stroke (width 0) (type default))
@@
     (stroke (width 0) (type default))
   )
+  (wire (pts (xy 34.29 135.89) (xy 41.275 135.89))
+    (stroke (width 0) (type default))
+  )
   (wire (pts (xy 31.115 189.865) (xy 38.1 189.865))
     (stroke (width 0) (type default))
@@
     (stroke (width 0) (type default))
   )
+  (wire (pts (xy 41.275 140.97) (xy 34.29 140.97))
+    (stroke (width 0) (type default))
+  )
   (wire (pts (xy 200.025 126.365) (xy 200.66 126.365))
     (stroke (width 0) (type default))
@@
     (stroke (width 0) (type default))
   )
+  (wire (pts (xy 78.74 138.43) (xy 78.74 128.905))
+    (stroke (width 0) (type default))
+  )
   (wire (pts (xy 332.74 83.185) (xy 343.535 83.185))
     (stroke (width 0) (type default))
@@
     (effects (font (size 1.55 1.55)) (justify right bottom))
   )
+  (text "U21D is wrong,\nit should be a OR Gate." (at 68.58 121.285 0)
+    (effects (font (size 1.27 1.27)) (justify left bottom))
+  )
   (text "CPR - Latches Date into int. Register\n~{MRC} - Clears int. Register\n~{OE} - Enables Output\nCPC - Clock Pulse for Counter"
     (at 302.895 167.64 0)
@@
     (effects (font (size 1.27 1.27)) (justify left bottom))
   )
+  (text "WP is LOW for RAM and\nHigh for ROM." (at 60.96 146.05 0)
+    (effects (font (size 1.27 1.27)) (justify left bottom))
+  )
   (text "B9\n" (at 23.495 230.505 0)
     (effects (font (size 1.55 1.55)) (justify right bottom))
@@
     (effects (font (size 1.27 1.27)) (justify left bottom))
   )
-  (text "B10 (B11 on F103)\nB2 (B10 on F103)" (at 60.325 200.025 0)
+  (text "B10 (B11 on F103)\nB2 (TRST on F103)" (at 60.325 200.025 0)
     (effects (font (size 1.27 1.27)) (justify left bottom))
   )
@@
     (effects (font (size 1.27 1.27)) (justify left bottom))
   )
-  (text "~{WP} is LOW for RAM and\nHigh for ROM." (at 76.835 121.285 0)
-    (effects (font (size 1.27 1.27)) (justify left bottom))
-  )
   (text "A7\nA6\nA5\nA4\nA3\nA2\nA1\nA0" (at 60.325 225.425 0)
     (effects (font (size 1.55 1.55)) (justify left bottom))
@@
     (effects (font (size 1.55 1.55)) (justify left bottom))
   )
-  (text "Chip Select Numbers:\n~{RAMWE0} - ~{RAMWE14} external Use for Peripherals\n~{RAMWE15} - RAMROM Card"
+  (text "Chip Select Numbers:\n~{RAMWE0} - ~{RAMWE13} external Use for Peripherals\n~{RAMWE14} - RAMROM Card Enable\n~{RAMWE15} - RAMROM Card RAMA Fill"
     (at 161.29 61.595 0)
     (effects (font (size 1.27 1.27)) (justify left bottom))
@@
     (effects (font (size 1.27 1.27)) (justify right bottom))
   )
-  (label "~{WP}" (at 66.04 114.3 0) (fields_autoplaced)
+  (label "WP" (at 66.04 114.3 0) (fields_autoplaced)
     (effects (font (size 1.27 1.27)) (justify left bottom))
   )
@@
     (effects (font (size 1.27 1.27)) (justify right bottom))
   )
+  (label "WP" (at 34.29 140.97 0) (fields_autoplaced)
+    (effects (font (size 1.27 1.27)) (justify left bottom))
+  )
   (label "A3" (at 93.345 53.975 0) (fields_autoplaced)
     (effects (font (size 1.27 1.27)) (justify left bottom))
@@
     (effects (font (size 1.27 1.27)) (justify left bottom))
   )
-  (label "B10" (at 59.055 197.485 180) (fields_autoplaced)
+  (label "TRST" (at 59.055 197.485 180) (fields_autoplaced)
     (effects (font (size 1.27 1.27)) (justify right bottom))
   )
+  (label "~{MWR}" (at 34.29 135.89 0) (fields_autoplaced)
+    (effects (font (size 1.27 1.27)) (justify left bottom))
+  )
   (label "CD2" (at 265.43 232.41 180) (fields_autoplaced)
     (effects (font (size 1.27 1.27)) (justify right bottom))
@@
     (effects (font (size 1.27 1.27)) (justify right bottom))
   )
-  (label "B10" (at 88.265 25.4 0) (fields_autoplaced)
+  (label "TRST" (at 88.265 25.4 0) (fields_autoplaced)
     (effects (font (size 1.27 1.27)) (justify left bottom))
   )
@@
     (effects (font (size 1.27 1.27)) (justify left bottom))
   )
-  (label "~{WP}" (at 283.21 73.025 180) (fields_autoplaced)
+  (label "WP" (at 283.21 73.025 180) (fields_autoplaced)
     (effects (font (size 1.27 1.27)) (justify right bottom))
   )
@@
     )
   )
+  (symbol (lib_id "power:+3V3") (at 56.515 128.27 0) (unit 1)
+    (in_bom yes) (on_board yes) (dnp no) (fields_autoplaced)
+    (property "Reference" "#PWR013" (at 56.515 132.08 0)
+      (effects (font (size 1.27 1.27)) hide)
+    )
+    (property "Value" "+3V3" (at 56.515 124.6942 0)
+      (effects (font (size 1.27 1.27)))
+    )
+    (property "Footprint" "" (at 56.515 128.27 0)
+      (effects (font (size 1.27 1.27)) hide)
+    )
+    (property "Datasheet" "" (at 56.515 128.27 0)
+      (effects (font (size 1.27 1.27)) hide)
+    )
+    (pin "1")
+    (instances
+      (project "RAMROM_512k_board"
+        (path "/2eaa3998-c9cb-43b1-9b23-df656c8158b0"
+          (reference "#PWR013") (unit 1)
+        )
+      )
+    )
+  )
   (symbol (lib_id "74xGxx:74AHC1G14") (at 217.17 240.03 0) (unit 1)
     (in_bom yes) (on_board yes) (dnp no) (fields_autoplaced)
@@
     )
   )
+  (symbol (lib_id "power:GND") (at 56.515 148.59 0) (unit 1)
+    (in_bom yes) (on_board yes) (dnp no) (fields_autoplaced)
+    (property "Reference" "#PWR041" (at 56.515 154.94 0)
+      (effects (font (size 1.27 1.27)) hide)
+    )
+    (property "Value" "GND" (at 56.515 153.0334 0)
+      (effects (font (size 1.27 1.27)))
+    )
+    (property "Footprint" "" (at 56.515 148.59 0)
+      (effects (font (size 1.27 1.27)) hide)
+    )
+    (property "Datasheet" "" (at 56.515 148.59 0)
+      (effects (font (size 1.27 1.27)) hide)
+    )
+    (pin "1")
+    (instances
+      (project "RAMROM_512k_board"
+        (path "/2eaa3998-c9cb-43b1-9b23-df656c8158b0"
+          (reference "#PWR041") (unit 1)
+        )
+      )
+    )
+  )
   (symbol (lib_id "Device:R_Small") (at 71.755 43.18 0) (unit 1)
     (in_bom yes) (on_board yes) (dnp no) (fields_autoplaced)
@@
         )
       )
+    )
+  )
+  (symbol (lib_id "74xGxx:74LVC1G32") (at 56.515 138.43 0) (unit 1)
+    (in_bom yes) (on_board yes) (dnp no) (fields_autoplaced)
+    (property "Reference" "U3" (at 67.8203 134.4128 0)
+      (effects (font (size 1.27 1.27)))
+    )
+    (property "Value" "74LVC1G32" (at 67.8203 136.837 0)
+      (effects (font (size 1.27 1.27)))
+    )
+    (property "Footprint" "Package_TO_SOT_SMD:SOT-23-5_HandSoldering" (at 56.515 138.43 0)
+      (effects (font (size 1.27 1.27)) hide)
+    )
+    (property "Datasheet" "http://www.ti.com/lit/sg/scyt129e/scyt129e.pdf" (at 56.515 138.43 0)
+      (effects (font (size 1.27 1.27)) hide)
+    )
+    (pin "1")
+    (pin "2")
+    (pin "3")
+    (pin "4")
+    (pin "5")
+    (instances
+      (project "RAMROM_512k_board"
+        (path "/2eaa3998-c9cb-43b1-9b23-df656c8158b0"
+          (reference "U3") (unit 1)
+        )
+      )

Commit message: python work
Parts:
- removed BT1: Battery_Cell, Battery:BatteryHolder_Keystone_103_1x20mm, symbol Device:Battery_Cell
- removed D2: BAT54C, Package_TO_SOT_SMD:SOT-23, symbol Diode:BAT54C
- J6: value STM32F411 -> STM32F401
Connections:
- net +3V3: now also C4.1, U4.11 (VDD), U4.33 (VDD)
- net WP: no longer U21.13
- net ~{CSRAM}: now also U1.19 (CE), U21.9; no longer U4.8 (~{CE})
- net ~{DATOE}: now also U21.1; no longer U21.4
- net ~{MRD}: now also U21.2; no longer U21.10, U21.5
- net ~{MWR}: no longer U21.12, U21.9
- net ~{RAMWE15}: now also U21.5; no longer U21.2
- net at U4.15 (~{WE}): now also U21.6; no longer U21.3
- net at U4.37 (~{OE}): now also U21.3; no longer U21.6
- net at U3.4: now also U21.4; no longer U21.1
- net at U21.8: now also U4.8 (~{CE}); no longer U1.19 (CE)
- net uA10 renamed ~{RAMCSOR}
- net ~{RAMCSOR}: now also U21.10
- no-connect marks 15 -> 17
Other:
- note added: "SCL SDA"
- note added: "U21C is wrong! Now ~{CSRAM} is for ~{CE} of U1."
- note added: "maybe use U21D for Select Override."
- moved on the sheet: U21A, U21B, U21C

Commit message: SYM1 & KIM1 work, RAM Board update
Parts:
- removed R10, R9: 10k, Resistor_SMD:R_1206_3216Metric_Pad1.30x1.75mm_HandSolder, symbol Device:R_Small
- added C7: 100n, Capacitor_SMD:C_1206_3216Metric, symbol Device:C_Small
- added J10, J11, J12, J13, J14, J5: ., Connector_PinHeader_2.00mm:PinHeader_1x01_P2.00mm_Vertical, symbol Connector_Generic:Conn_01x01
- added R3, R4, R5, R6: 3k3, Resistor_SMD:R_1206_3216Metric, symbol Device:R_Small
- added RN1, RN2: 10k, Resistor_THT:R_Array_SIP11, symbol Device:R_Network10
- added U11: DS1085, Package_SO:SOIC-8_3.9x4.9mm_P1.27mm, symbol my_ics_new:DS1085
- added U13: 74LVC125, Package_SO:SOIC-14_3.9x8.7mm_P1.27mm, symbol 74xx:74LS125
- R7, R8: footprint Resistor_SMD:R_1206_3216Metric_Pad1.30x1.75mm_HandSolder -> Resistor_SMD:R_1206_3216Metric
Connections:
- net B2 is gone; now on net ~{DATOE}: J6.36 (Pin_36)
- net +3V3: now also R7.1, R8.1, C7.1, R3.1, R4.1, R5.1, R6.1, U11.3 (Vcc), U13.14 (VCC)
- net A0: now also RN1.11 (R10)
- net A1: now also RN2.11 (R10)
- net A10: now also RN1.6 (R5)
- net A11: now also RN2.6 (R5)
- net A12: now also RN1.5 (R4)
- net A13: now also RN2.5 (R4)
- net A14: now also RN1.4 (R3)
- net A15: now also RN2.4 (R3)
- net A16: now also RN1.3 (R2); no longer R7.1
- net A17: now also RN2.3 (R2); no longer R8.1
- net A18: now also RN1.2 (R1)
- net A19: now also RN2.2 (R1)
- net A2: now also RN1.10 (R9)
- net A3: now also RN2.10 (R9)
- net A4: now also J6.30 (Pin_30), RN1.9 (R8)
- net A5: now also RN2.9 (R8)
- net A6: now also RN1.8 (R7)
- net A7: now also RN2.8 (R7)
- net A8: now also RN1.7 (R6)
- net A9: now also RN2.7 (R6)
- net CLKF: now also U13.8
- net CLKS: now also U13.11
- net GND: now also C7.2, RN1.1 (common), RN2.1 (common), U11.4 (GND), U13.1, U13.10, U13.13, U13.4, U13.7 (GND); no longer R7.2, R8.2
- net ~{DATOE}: no longer J6.30 (Pin_30)
- net ~{MRD}: now also R8.2
- net ~{MWR}: now also R7.2
- net B6 renamed SCL
- net SCL: now also R3.2, U11.8 (SCL)
- net B7 renamed SDA
- net SDA: now also R4.2, U11.7 (SDA)
- net B8 renamed CTRL1
- net CTRL1: now also J10.1 (Pin_1), R6.2, U11.6 (CTRL1)
- new net: J5.1 (Pin_1), R5.2, U11.5 (CTRL0)
- new net: J11.1 (Pin_1), U13.3
- new net: J13.1 (Pin_1), U13.2
- new net: J14.1 (Pin_1), U13.5
- new net: J12.1 (Pin_1), U13.6
- new net CLKF#: U11.2 (OUT0), U13.9
- new net CLKS#: U11.1 (OUT1), U13.12
Other:
- note added: "ATTENTION: ~{DATOE} changed from A4 to B2!"
- note added: "Address Counter"
- note added: "B10 (B11 on F103) B2 (B10 on F103)"
- note added: "B6 (SCL) B7 (SDA) B8"
- note added: "Chip Select for RAM and writeprotect for ROM."
- note added: "Clock Generator"
- note added: "Data read and write from main RAM."
- note added: "STM32F401 microcontroller"
- note added: "Solder the SIP in the holes of J3."
- note added: "Write Pulse for the Peripheral chips."
- note removed: "B10 (B11 on F103) B2 (TRST on F103)"
- note removed: "SCL SDA"
- moved on the sheet: C1, C10, C2, C3, C5, C6, C8, C9, H1, H2, H3, H4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

Commit message: Documentation update
Parts:
- removed J7, J9: ., Connector_PinHeader_2.00mm:PinHeader_1x01_P2.00mm_Vertical, symbol Connector_Generic:Conn_01x01
- added C11: 100n, Capacitor_SMD:C_1206_3216Metric, symbol Device:C_Small
Connections:
- net +3V3: now also C11.1
- net A4: no longer J6.30 (Pin_30)
- net GND: now also C11.2
- net MOSI: now also U2.8; no longer U10.14 (SER), U7.14 (SER)
- net SCK: now also U2.3, U2.6; no longer U10.11 (SRCLK), U12.2, U2.8, U7.11 (SRCLK), U8.2, U9.2 (CP)
- net uMOSI: now also U10.14 (SER), U2.9, U7.14 (SER)
- net uSCK: now also U10.11 (SRCLK), U12.2, U2.2, U2.5, U7.11 (SRCLK), U8.2, U9.2 (CP); no longer U2.9
- net ~{uMRD}: no longer U2.5
- net ~{uMWR}: no longer U2.2
- net UMISO renamed uMISO
- new net uA4: J6.30 (Pin_30)
Other:
- moved on the sheet: U21E, U2A, U2B, U2C, U2D
