File: Splitter Board/schematic/SplitterBoard/SplitterBoard.kicad_pcb (KiCad board)
At the start: 2 copper layers, 100 x 100 mm, 23 parts, among them J1 BUS-Master, J10 GND, J11 Conn_01x03, J12 Conn_01x03, J2 BUS-Master, J3 BUS-Master-BO, J4 BUS-Master-BO, J5 BUS-Angled, J6 BUS-Angled, J7 Conn_01x21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

Commit message: 6809 Board done, Splitter Board new, RAMROM512k new
Parts:
- added J13: Conn_01x01, Connector_PinHeader_2.00mm:PinHeader_1x01_P2.00mm_Vertical, F.Cu at (180.2, 73.9)
- added J14: Conn_01x01, Connector_PinHeader_2.00mm:PinHeader_1x01_P2.00mm_Vertical, F.Cu at (180.2, 69.1)
- added J15: Conn_01x02, Connector_PinHeader_2.54mm:PinHeader_1x02_P2.54mm_Vertical, F.Cu at (194.5, 79.8)
- added J16: Conn_01x01, Connector_PinHeader_2.00mm:PinHeader_1x01_P2.00mm_Vertical, F.Cu at (183.3, 73.9)
- added J17: Conn_01x01, Connector_PinHeader_2.00mm:PinHeader_1x01_P2.00mm_Vertical, F.Cu at (179.7, 79.4)
- added JP3: ., Jumper:SolderJumper-3_P1.3mm_Open_Pad1.0x1.5mm_NumberLabels, B.Cu at (176.0, 80.7)
- added JP4: ., Jumper:SolderJumper-3_P1.3mm_Open_Pad1.0x1.5mm_NumberLabels, B.Cu at (184.8, 65.1)
- added JP5: ., Jumper:SolderJumper-3_P1.3mm_Open_Pad1.0x1.5mm_NumberLabels, B.Cu at (182.2, 65.1)
- moved JP2 12.3 mm to (112.0, 66.8)
Connections:
- JP1 pad 2: /~{extCS} -> Net-(JP1-C)
- U1 pad 1: GND -> /OUT/~{IN}
- U2 pad 1: GND -> /OUT/~{IN}
- U4 pad 1: GND -> /OUT/~{IN}
Routing:
- net /OUT/~{IN}: track 0.00 -> 85.0 mm, vias 0 -> 1
- net Net-(JP1-C): track 0.00 -> 57.4 mm, vias 0 -> 2
- net /~{extCS}: track 139.6 -> 91.5 mm, vias 1 -> 0
- net GND: track 501.0 -> 524.5 mm, vias 2 -> 5
- net /~{CS_ext}: track 0.00 -> 22.9 mm
- net /VBuffer: track 73.4 -> 89.6 mm, vias 2 -> 3
- net +3V3: track 153.0 -> 162.8 mm
- net /PHI1_e: track 97.1 -> 92.3 mm
- net /A19s: track 73.7 -> 77.2 mm, vias 0 -> 1
- net +5V: track 288.7 -> 289.9 mm
- net /PHI2_e: track 97.7 -> 96.6 mm
- net /~{RAMWE13}: track 92.7 -> 91.7 mm
- net /A15s: track 79.3 -> 78.3 mm
- net /A10s: track 85.8 -> 85.1 mm
- net /~{IOWR}: track 97.7 -> 97.0 mm
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Other:
- board text added: "*Unicomp v2* Splitter Board v1.1"
- board text removed: "*Unicomp v2* Splitter Board v1.0"
