File: Splitter Board/schematic/SplitterBoard/SplitterBoard.kicad_sch (KiCad schematic)
At the start: 23 parts, among them J1 BUS-Master, J10 GND, J11 Conn_01x03, J12 Conn_01x03, J2 BUS-Master, J3 BUS-Master-BO, J4 BUS-Master-BO, J5 BUS-Angled, J6 BUS-Angled, J7 Conn_01x21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

Commit message: 6809 Board done, Splitter Board new, RAMROM512k new
Parts:
- added J13, J14, J16, J17: Conn_01x01, Connector_PinHeader_2.00mm:PinHeader_1x01_P2.00mm_Vertical, symbol Connector_Generic:Conn_01x01
- added J15: Conn_01x02, Connector_PinHeader_2.54mm:PinHeader_1x02_P2.54mm_Vertical, symbol Connector_Generic:Conn_01x02
- added JP3, JP4, JP5: ., Jumper:SolderJumper-3_P1.3mm_Open_Pad1.0x1.5mm_NumberLabels, symbol Jumper:Jumper_3_Bridged12
- renumbered JP29 to JP2
Connections:
- net GND: now also JP4.1 (A), JP5.1 (A); no longer U1.1 (A->B), U2.1 (A->B), U4.1 (A->B)
- net VBuffer: now also JP4.3 (B), JP5.3 (B)
- net ~{extCS}: now also J14.1 (Pin_1), JP3.2 (C), JP4.2 (C); no longer JP1.2 (C)
- new net: JP1.2 (C), JP3.1 (A)
- new net OUT/~{IN}: J13.1 (Pin_1), J15.1 (Pin_1), J16.1 (Pin_1), JP5.2 (C), U1.1 (A->B), U2.1 (A->B), U4.1 (A->B)
- new net ~{CS_ext}: J15.2 (Pin_2), J17.1 (Pin_1), JP3.3 (B)
Other:
- moved on the sheet: JP1
