File: CPLD_board/schematic/cpld_board_max2/cpld_board_max2.kicad_pcb (KiCad board)
At the start: 2 copper layers, 100 x 100 mm, 56 parts, among them J1 BUS-Master, J10 GND, J11 Conn_01x02, J12 RX_TX, J13 Conn_02x05_Odd_Even, J14 ., J15 Conn_01x02, J16 ., J17 ., J18 ., J19 ., J2 BUS-Master, J20 ., J22 ., J23 ., J24 ., J25 ., J26 ., J27 ., J28 ., J29 ., J3 BUS-Master-BO, J4 BUS-Master-BO, J5 BUS-Angled, J6 STM32F401, J7 Micro_SD_Card_Det2, J8 USB_A, J9 Raspberry_Pi_2_3, SW1 SW_Push, SW2 SW_Push, SW3 SW_Push, SW4 SW_Push, U1 ebay MAX II board, U2 74HC245, U3 IS61LV256AL-10JL

Commit message: olimex scripts updated
Parts:
- H1, H2, H3, H4, H5, H6, H7, H8: value MountingHole -> MountinSREDole
- J13: moved to B.Cu
- J5: value BUS-Angled -> BUS-AnHSYNCed
- J8: value USB_A -> USB_A_Molex_67643
- moved J13 10.2 mm to (161.0, 72.8)
Connections:
- net /BH renamed /RED
- net /BH# renamed /RED#
- net /BL renamed /VSYNC
- net /C15 renamed /BLU
- net /GH renamed /Q1
- net /GL renamed /HSYNC
- net /GL# renamed /HSYNC#
- net /HSYN renamed /GRN
- J13 pad 1: /VSYN# -> GND
- J13 pad 10: /RH# -> +3V3
- J13 pad 2: +3V3 -> /SGRN#
- J13 pad 3: /HSYN# -> /SRED#
- J13 pad 4: /BL# -> /SBLU#
- J13 pad 7: /GH# -> /GRN#
- J13 pad 8: /RL# -> /VSYNC#
- J13 pad 9: GND -> /BLU#
- U2 pad 2: /VSYN# -> /BLU#
- U2 pad 3: /BL# -> /VSYNC#
- U2 pad 4: /HSYN# -> /GRN#
- U2 pad 7: /RL# -> /SBLU#
- U2 pad 8: /GH# -> /SRED#
- U2 pad 9: /RH# -> /SGRN#
Routing:
- net /VSYNC#: track 0.00 -> 6.82 mm
- net /SGRN#: track 0.00 -> 6.82 mm
- net /SBLU#: track 0.00 -> 6.82 mm
- net /RL#: track 6.82 -> 0.00 mm
- net /RH#: track 6.82 -> 0.00 mm
- net /BL#: track 6.82 -> 0.00 mm
- net /VSYN#: track 3.77 -> 0.00 mm
- net /HSYN#: track 3.77 -> 0.00 mm
- net /GRN#: track 0.00 -> 3.77 mm
- net /BLU#: track 0.00 -> 3.77 mm
- net /SRED#: track 0.00 -> 3.77 mm
- net /GH#: track 3.77 -> 0.00 mm
