File: CPLD_board/schematic/cpld_board_max2/cpld_board_max2.kicad_sch (KiCad schematic)
At the start: 56 parts, among them J1 BUS-Master, J10 GND, J11 Conn_01x02, J12 RX_TX, J13 Conn_02x05_Odd_Even, J14 ., J15 Conn_01x02, J16 ., J17 ., J18 ., J19 ., J2 BUS-Master, J20 ., J21 ., J22 ., J23 ., J24 ., J25 ., J26 ., J27 ., J28 ., J29 ., J3 BUS-Master-BO, J4 BUS-Master-BO, J5 BUS-Angled, J6 STM32F401, J7 Micro_SD_Card_Det2, J8 USB_A_Molex_67643, J9 Raspberry_Pi_2_3, SW1 SW_Push, SW2 SW_Push, SW3 SW_Push, SW4 SW_Push, U1 ebay MAX II board, U2 74HC245, U3 IS61LV256AL-10JL

Commit message: olimex scripts updated
Parts:
- H1, H2, H3, H4, H5, H6, H7, H8: value MountingHole -> MountinSREDole
- J5: value BUS-Angled -> BUS-AnHSYNCed
Connections:
- net +3V3: now also J13.10 (Pin_10); no longer J13.2 (Pin_2)
- net GND: now also J13.1 (Pin_1); no longer J13.9 (Pin_9)
- net BH renamed RED
- net BH# renamed RED#
- net BL renamed VSYNC
- net BL# renamed SBLU#
- net SBLU#: now also U2.7 (A5); no longer U2.3 (A1)
- net C15 renamed BLU
- net GH renamed Q1
- net GH# renamed GRN#
- net GRN#: now also U2.4 (A2); no longer U2.8 (A6)
- net GL renamed HSYNC
- net GL# renamed HSYNC#
- net HSYN renamed GRN
- net HSYN# renamed SRED#
- net SRED#: now also U2.8 (A6); no longer U2.4 (A2)
- net RH# renamed SGRN#
- net SGRN#: now also J13.2 (Pin_2); no longer J13.10 (Pin_10)
- net RL# renamed VSYNC#
- net VSYNC#: now also U2.3 (A1); no longer U2.7 (A5)
- net VSYN# renamed BLU#
- net BLU#: now also J13.9 (Pin_9); no longer J13.1 (Pin_1)
Other:
- note added: "CGA/EGA Pin: - 9 8 7 6"
- note added: "CGA/EGA Pin: 5 4 3 2 1"
- moved on the sheet: J13
