File: 6803_Board/6803_board/6803_board.kicad_pcb (KiCad board)
At the start: 2 copper layers, 100 x 100 mm, 71 parts, among them J1 BUS, J10 Conn_01x01, J11 Conn_01x01, J12 Conn_01x01, J13 Conn_01x01, J14 Conn_01x01, J15 Conn_01x01, J16 ., J17 ., J18 .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

Commit message: MC3 Computer update
Routing:
- net /~{RST}: track 6.96 -> 89.7 mm, vias 0 -> 1
- net +5V: track 229.8 -> 219.7 mm
- net /Buffers/VBuffer: track 204.3 -> 197.2 mm
- net +3V3: track 192.9 -> 189.6 mm
