File: 6502_6802 Board v2/schematic/6303R_PLCC_Addon/6303_PLCC.kicad_pcb (KiCad board)
At the start: 2 copper layers, 68 x 49.8 mm, 21 parts, among them J1 Conn_02x08_Odd_Even, J2 ., J3 ., J4 ., J5 ., J6 ., U1 HD6303RCP, U2 74LS573, U3 MC6802

Commit message: some work on the CPU Adapter Boards
Connections:
- U1 pad 10: (no net) -> unconnected-(U1-~{STBY}-Pad10)
Changed lines of the file:
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@@
   (net 65 "unconnected-(U1-Pad46)")
   (net 66 "unconnected-(U1-Pad47)")
+  (net 67 "unconnected-(U1-~{STBY}-Pad10)")
   (footprint "Connector_PinHeader_2.54mm:PinHeader_2x08_P2.54mm_Horizontal" (layer "F.Cu")
     (at 167.132 71.374 180)
@@
       (stroke (width 0.1) (type solid)) (layer "F.Fab"))
     (pad "1" thru_hole rect (at 0 0 90) (size 1.6 1.6) (drill 0.8) (layers "*.Cu" "*.Mask")
-      (net 2 "GND") (pinfunction "VSS") (pintype "power_in"))
+      (net 2 "GND") (pinfunction "VSS") (pintype "passive"))
     (pad "2" thru_hole oval (at 0 2.54 90) (size 1.6 1.6) (drill 0.8) (layers "*.Cu" "*.Mask")
       (net 54 "/~{HALT}") (pinfunction "~{HALT}") (pintype "input"))
@@
     (pad "9" smd rect (at -9.1325 -6.35 90) (size 1.925 0.7) (layers "F.Cu" "F.Paste" "F.Mask")
       (net 8 "/~{RST}") (pinfunction "~{RST}") (pintype "input"))
-    (pad "10" smd rect (at -9.1325 -5.08 90) (size 1.925 0.7) (layers "F.Cu" "F.Paste" "F.Mask"))
+    (pad "10" smd rect (at -9.1325 -5.08 90) (size 1.925 0.7) (layers "F.Cu" "F.Paste" "F.Mask")
+      (net 67 "unconnected-(U1-~{STBY}-Pad10)") (pinfunction "~{STBY}") (pintype "input"))
     (pad "11" smd rect (at -9.1325 -3.81 90) (size 1.925 0.7) (layers "F.Cu" "F.Paste" "F.Mask")
       (net 3 "/P20") (pinfunction "P20/Tin") (pintype "bidirectional"))
