File: 6502_6802 Board v2/schematic/6303R_PLCC_Addon/6303_PLCC.kicad_sch (KiCad schematic)
At the start: 21 parts, among them J1 Conn_02x08_Odd_Even, J2 ., J3 ., J4 ., J5 ., J6 ., U1 HD6303RCP, U2 74LS573, U99 MC6802

Commit message: some work on the CPU Adapter Boards
Other:
- note added: "HD6303 needes Pin2 open!"
- note added: "This does NOT work for HD6303!"
- note added: "forgot ~{STBY} Pullup!"
Changed lines of the file:
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@@
     (stroke (width 0) (type default))
   )
+  (text "forgot ~{STBY} Pullup!" (at 39.37 58.42 0)
+    (effects (font (size 1.27 1.27)) (justify left bottom))
+  )
+  (text "This does NOT work for HD6303!" (at 55.245 176.53 0)
+    (effects (font (size 1.27 1.27)) (justify left bottom))
+  )
   (text "E is Clock in on 6803E!" (at 114.935 107.315 0)
+    (effects (font (size 1.27 1.27)) (justify left bottom))
+  )
+  (text "HD6303 needes\nPin2 open!" (at 63.5 95.25 0)
     (effects (font (size 1.27 1.27)) (justify left bottom))
   )
@@
     (pin "13")
     (pin "12")
-    (instances
-      (project "6303_PLCC"
+    (pin "10")
+    (instances
+      (project "6303_PLCC"
