File: LCDBoard/Unicomp_LCD_Board/Unicomp_LCD_Board.kicad_pcb (KiCad board)
At the start: 2 copper layers, 88 x 85 mm, 69 parts, among them J1 BUS, J10 ., J11 ., J12 ., J13 ., J14 ., J15 NMI, J16 ., J17 ., J18 ., J19 ., J2 ~{RAMCE}, J20 ., J21 ., J22 ., J23 ., J24 ., J25 KBD_CLK, J26 KBD_CLK, J27 ., J28 ~{RST}, J29 ~{RST}, J3 ., J30 P57, J31 READY, J32 Keyb, J33 ~{STBY}, J4 ., J5 ., J6 ., J7 P57, J8 ., J9 ., Q1 BC327, SW1 ON, U1 NHD-0420H1Z, U2 4011, U3 4081, U4 Recom RMSR-0505, U5 4013, U6 4040, U7 NHD-0420H1Z

Commit message: some work on the CPU Adapter Boards
Parts:
- J22: value . -> LCD_E
- R6: value 47k -> 1k
Routing:
- added copper zone on B.Cu, net GND
Changed lines of the file:
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@@
         (effects (font (size 1 1) (thickness 0.15)))
     )
-    (fp_text value "P57" (at 0 2.06) (layer "F.Fab")
+    (fp_text value "P57" (at 0.988 4.084) (layer "F.Fab")
         (effects (font (size 1 1) (thickness 0.15)))
     )
@@
         (effects (font (size 1 1) (thickness 0.15)))
     )
-    (fp_text value "READY" (at 0 2.06) (layer "F.Fab")
+    (fp_text value "READY" (at -0.964 4.434) (layer "F.Fab")
         (effects (font (size 1 1) (thickness 0.15)))
     )
@@
         (effects (font (size 1 1) (thickness 0.15)))
     )
-    (fp_text value "." (at 0 2.06) (layer "F.Fab")
+    (fp_text value "LCD_E" (at 0 2.06) (layer "F.Fab")
         (effects (font (size 1 1) (thickness 0.15)))
     )
@@
         (effects (font (size 1 1) (thickness 0.15)) (justify mirror))
     )
-    (fp_text value "47k" (at 0 -1.82) (layer "B.Fab")
+    (fp_text value "1k" (at 0 -1.82) (layer "B.Fab")
         (effects (font (size 1 1) (thickness 0.15)) (justify mirror))
     )
@@
   (gr_rect (start 70 22) (end 158 107)
     (stroke (width 0.1) (type default)) (fill none) (layer "Edge.Cuts"))
-  (gr_text "PSION Organizer I\nR. OFFNER\n2024" (at 81.026 41.91 90) (layer "B.Cu")
+  (gr_text "PSION Organizer I\nR. OFFNER\n2024" (at 81.026 41.91 90) (layer "B.Cu" knockout)
     (effects (font (size 1.5 1.5) (thickness 0.3) bold) (justify left bottom mirror))
   )
@@
   (segment (start 73.66 86.868) (end 71.374 89.154) (width 0.4) (layer "B.Cu") (net 38))
   (segment (start 105.220233 104.648) (end 148.492 104.648) (width 0.4) (layer "B.Cu") (net 38))
-  (segment (start 82.356119 36.636119) (end 79.756 34.036) (width 0.4) (layer "B.Cu") (net 38))
   (segment (start 87.376 101.3845) (end 87.45125 101.30925) (width 0.4) (layer "B.Cu") (net 38))
   (segment (start 152.908 42.926) (end 152.908 29.718) (width 0.4) (layer "B.Cu") (net 38))
@@
   (segment (start 152.395 98.205) (end 150.6 100) (width 0.4) (layer "B.Cu") (net 38))
   (segment (start 91.186 86.868) (end 73.66 86.868) (width 0.4) (layer "B.Cu") (net 38))
-  (segment (start 79.756 72.644) (end 82.356119 70.043881) (width 0.4) (layer "B.Cu") (net 38))
   (segment (start 84.6205 102.87) (end 84.582 102.87) (width 0.4) (layer "B.Cu") (net 38))
   (segment (start 151.384 44.958) (end 151.384 57.658) (width 0.4) (layer "B.Cu") (net 38))
@@
   (segment (start 132.08 85.09) (end 133.858 85.09) (width 0.4) (layer "B.Cu") (net 38))
   (segment (start 146.558 61.214) (end 146.558 62.992) (width 0.4) (layer "B.Cu") (net 38))
-  (segment (start 82.356119 70.043881) (end 82.356119 36.636119) (width 0.4) (layer "B.Cu") (net 38))
   (segment (start 119.38 68.072) (end 129.54 57.912) (width 0.4) (layer "B.Cu") (net 38))
   (segment (start 118.364 82.042) (end 129.032 82.042) (width 0.4) (layer "B.Cu") (net 38))
@@
   (segment (start 152.4 29.21) (end 131.064 29.21) (width 0.4) (layer "B.Cu") (net 38))
   (segment (start 91.58225 92.31575) (end 93.472 90.426) (width 0.4) (layer "B.Cu") (net 38))
+  (segment (start 81.8 70.6) (end 81.8 36.08) (width 0.4) (layer "B.Cu") (net 38))
   (segment (start 151.13 44.704) (end 152.908 42.926) (width 0.4) (layer "B.Cu") (net 38))
   (segment (start 93.472 90.426) (end 93.472 88.646) (width 0.4) (layer "B.Cu") (net 38))
   (segment (start 147.066 60.706) (end 146.558 61.214) (width 0.4) (layer "B.Cu") (net 38))
   (segment (start 103.63 98.296) (end 103.63 103.057767) (width 0.4) (layer "B.Cu") (net 38))
+  (segment (start 79.756 72.644) (end 81.8 70.6) (width 0.4) (layer "B.Cu") (net 38))
   (segment (start 152.395 83.053) (end 152.395 85.08) (width 0.4) (layer "B.Cu") (net 38))
   (segment (start 151.384 58.42) (end 149.098 60.706) (width 0.4) (layer "B.Cu") (net 38))
+  (segment (start 81.8 36.08) (end 79.756 34.036) (width 0.4) (layer "B.Cu") (net 38))
   (segment (start 144.78 62.992) (end 146.558 62.992) (width 0.4) (layer "B.Cu") (net 38))
   (segment (start 89.26775 102.47575) (end 88.1765 101.3845) (width 0.4) (layer "B.Cu") (net 38))
@@
   (segment (start 126.492 48.394) (end 126.492 47.244) (width 0.4) (layer "B.Cu") (net 98))
   (segment (start 128.524 50.426) (end 126.492 48.394) (width 0.4) (layer "B.Cu") (net 98))
+  (zone (net 38) (net_name "GND") (layer "B.Cu") (hatch edge 0.5)
+    (connect_pads (clearance 0.5))
+    (min_thickness 0.25) (filled_areas_thickness no)
+    (fill yes (thermal_gap 0.5) (thermal_bridge_width 0.5))
+    (polygon
+      (pts
+        (xy 159.35 20.9)
+        (xy 159.5 107.6)
+        (xy 68.5 107.45)
+        (xy 68.85 21.25)
+      )
+    )
+  )
 )
