File: LCDBoard/Unicomp_LCD_Board/Unicomp_LCD_Board.kicad_sch (KiCad schematic)
At the start: 69 parts, among them J1 BUS, J10 ., J11 ., J12 ., J13 ., J14 ., J15 NMI, J16 ., J17 ., J18 ., J19 ., J2 ~{RAMCE}, J20 ., J21 ., J22 ., J23 ., J24 ., J25 KBD_CLK, J26 KBD_CLK, J27 ., J28 ~{RST}, J29 ~{RST}, J3 ., J30 P57, J31 READY, J32 Keyb, J33 ~{STBY}, J4 ., J5 ., J6 ., J7 P57, J8 ., J9 ., Q1 BC327, SW1 ON, U1 NHD-0420H1Z, U2 4011, U3 4081, U4 Recom RMSR-0505, U5 4013, U6 4040, U7 NHD-0420H1Z

Commit message: some work on the CPU Adapter Boards
Parts:
- added U8, U9: 74LS00, symbol 74xx:74LS00
- J22: value . -> LCD_E
- R6: value 47k -> 1k
Connections:
- net A14: now also U8.1
- net at U2.11, U3.13: now also U8.11
- net at J15.1 (Pin_1), U2.12: now also U8.12
- net at J23.1 (Pin_1), U2.13: now also U8.13
- net at D1.2 (A), R1.2, U2.2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: now also U8.2
- net at J2.1 (Pin_1), U2.3: now also U8.3
Other:
- note added: "<-Done"
- note added: "<-changed"
- note added: "Done->"
- moved on the sheet: J6
