File: Z80_Board/z80_schematics/buffers.kicad_sch (KiCad schematic)
At the start: 23 parts, among them J10 Conn_01x01, J11 Conn_01x01, J12 Conn_01x01, J13 Conn_01x01, J14 Conn_01x01, J15 Conn_01x01, J30 Conn_01x06, J31 Conn_01x06, U2 SN74LVC245ANSR, U3 SN74LVC245ANSR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

Commit message: Z80 added
Parts:
- removed J12, J13, J14, J15: Conn_01x01, Connector_PinHeader_1.27mm:PinHeader_1x01_P1.27mm_Vertical, symbol Connector_Generic:Conn_01x01
- added R12, R8: 10k, Resistor_SMD:R_1206_3216Metric_Pad1.30x1.75mm_HandSolder, symbol Device:R_Small
- R10, R11, R9: value 1k -> 10k
- renumbered U6 to U21
Connections:
- net PHI2 is gone; now on an unnamed net: U9.2
- net PHI2_e is gone; now on an unnamed net: U9.3
- net GND: no longer U9.4
- net R/~{W}: now also U8.2; no longer U8.5
- net R/~{W}_e: now also U8.3; no longer U8.6
- net VBuffer: now also R12.1, R8.1
- net ~{AOE}: now also U9.4
- net PH1: now reaches U9.11
- net PH2: now reaches U9.8
- net at J10.1 (Pin_1): no longer U8.3
- net PH2c: now reaches U9.9
- net PH1c: now reaches U9.12
- net at J11.1 (Pin_1): no longer U8.2
- net PHI0c renamed PHI0_c
- net PHI1 renamed ~{IORDc}
- net PHI1_e renamed ~{IORD}
- net ~{IORD}: now also R12.2
- net ~{PHI0c} renamed ~{PHI0_c}
- net ~{RDc} renamed ~{MRDc}
- net ~{WRc} renamed ~{MWRc}
- new net ~{IOWRc}: U8.5
- new net ~{IOWR}: R8.2, U8.6
Other:
- note removed: "maybe consider ~{MWR} and ~{MRD} NOT High-Z with AOE. Is this really necessary?"
- company: 100% Offner -> (none)
- title: Unicomp v2 - 6502 6802 Board -> (none)
